Commit message: fix: initial_value match spawn pose, startup ramp, lighter masses
- URDF: initial_value=0/0/-0.3 to match Gazebo spawn, reduced leg masses,
  effort 40Nm, softer contact params, removed problematic XML comment
- trot_node: 2s smoothstep startup ramp from spawn pose to standing
- launch: removed -J flags and pause mode, trot_node starts immediately
- PID: reduced gains for smoother control
- Robot still unstable at spawn - needs further investigation

Co-Authored-By: Claude Opus 4.6 <noreply@anthropic.com>

File: src/dog_description/urdf/dog.urdf.xacro (robot description, xacro)
@@ -5,22 +5,18 @@
     <xacro:property name="trunk_w" value="0.18"/>
     <xacro:property name="trunk_h" value="0.1"/>
-    <xacro:property name="trunk_m" value="6.0"/>
+    <xacro:property name="trunk_m" value="5.0"/>
     <xacro:property name="hip_l" value="0.06"/>
-    <xacro:property name="hip_m" value="0.2"/>
+    <xacro:property name="hip_m" value="0.15"/>
     <xacro:property name="hip_r" value="0.02"/>
     <xacro:property name="thigh_l" value="0.144"/>
     <xacro:property name="shin_l" value="0.1525"/>
-    <xacro:property name="leg_m" value="0.6"/>
+    <xacro:property name="thigh_m" value="0.3"/>
+    <xacro:property name="shin_m" value="0.15"/>
     <xacro:property name="leg_r" value="0.02"/>
-    <xacro:property name="foot_r" value="0.025"/>
-    <!-- Начальная поза стойки: IK(x=0, z=-0.22) -->
-    <!-- thigh=0.76 rad, shin=-1.47 rad => нога опущена на 0.22м ниже бедра -->
-    <xacro:property name="init_thigh" value="0.76"/>
-    <xacro:property name="init_shin" value="-1.47"/>
+    <xacro:property name="foot_r" value="0.02"/>
     <!-- ==================== MATERIALS ==================== -->
     <material name="black"><color rgba="0.1 0.1 0.1 1"/></material>
     <material name="grey"><color rgba="0.6 0.6 0.6 1"/></material>
     <!-- ==================== INERTIA MACROS ==================== -->
-    <!-- Box inertia (CoM в центре box) -->
     <xacro:macro name="box_inertia" params="m l w h">
         <inertial>
@@ -31,5 +27,4 @@
         </inertial>
     </xacro:macro>
-    <!-- Cylinder inertia со смещённым центром масс -->
     <xacro:macro name="cylinder_inertia_offset" params="m r h ox oy oz">
         <inertial>
@@ -63,7 +58,7 @@
             <mu1>1.5</mu1>
             <mu2>1.5</mu2>
-            <kp>100000.0</kp>
-            <kd>100.0</kd>
-            <minDepth>0.001</minDepth>
+            <kp>50000.0</kp>
+            <kd>50.0</kd>
+            <minDepth>0.002</minDepth>
         </gazebo>
     </xacro:macro>
@@ -75,6 +70,6 @@
             <origin xyz="${side_x * trunk_l/2} ${side_y * trunk_w/2} 0" rpy="0 0 0"/>
             <axis xyz="1 0 0"/>
-            <limit lower="-0.5" upper="0.5" effort="20" velocity="10"/>
-            <dynamics damping="1.0" friction="0.3"/>
+            <limit lower="-0.5" upper="0.5" effort="40" velocity="10"/>
+            <dynamics damping="0.5" friction="0.1"/>
         </joint>
         <link name="${prefix}_hip">
@@ -92,6 +87,6 @@
             <origin xyz="0 ${side_y * hip_l} 0" rpy="0 0 0"/>
             <axis xyz="0 1 0"/>
-            <limit lower="-0.5" upper="2.5" effort="20" velocity="10"/>
-            <dynamics damping="1.0" friction="0.3"/>
+            <limit lower="-0.5" upper="2.5" effort="40" velocity="10"/>
+            <dynamics damping="0.5" friction="0.1"/>
         </joint>
         <link name="${prefix}_thigh">
@@ -103,7 +98,7 @@
             <collision>
                 <origin xyz="0 0 ${-thigh_l/2}"/>
-                <geometry><cylinder radius="${leg_r}" length="${thigh_l - 0.04}"/></geometry>
+                <geometry><cylinder radius="${leg_r}" length="${thigh_l}"/></geometry>
             </collision>
-            <xacro:cylinder_inertia_offset m="${leg_m}" r="${leg_r}" h="${thigh_l}"
+            <xacro:cylinder_inertia_offset m="${thigh_m}" r="${leg_r}" h="${thigh_l}"
                 ox="0" oy="0" oz="${-thigh_l/2}"/>
         </link>
@@ -113,6 +108,6 @@
             <origin xyz="0 0 ${-thigh_l}" rpy="0 0 0"/>
             <axis xyz="0 1 0"/>
-            <limit lower="-2.7" upper="-0.3" effort="20" velocity="10"/>
-            <dynamics damping="1.0" friction="0.3"/>
+            <limit lower="-2.7" upper="-0.3" effort="40" velocity="10"/>
+            <dynamics damping="0.5" friction="0.1"/>
         </joint>
         <link name="${prefix}_shin">
@@ -131,5 +126,5 @@
                 <geometry><sphere radius="${foot_r}"/></geometry>
             </collision>
-            <xacro:cylinder_inertia_offset m="${leg_m}" r="${leg_r*0.8}" h="${shin_l}"
+            <xacro:cylinder_inertia_offset m="${shin_m}" r="${leg_r*0.8}" h="${shin_l}"
                 ox="0" oy="0" oz="${-shin_l/2}"/>
         </link>
@@ -142,7 +137,8 @@
     <xacro:dog_leg prefix="rear_right"  side_x="-1" side_y="-1"/>
     <!-- ==================== ROS2 CONTROL ==================== -->
+    <!-- initial_value MUST match the physical spawn pose (thigh=0, shin=-0.3) -->
     <ros2_control name="GazeboSystem" type="system">
         <hardware><plugin>gazebo_ros2_control/GazeboSystem</plugin></hardware>
-        <xacro:macro name="init_pos" params="name t s">
+        <xacro:macro name="init_pos" params="name">
             <joint name="${name}_hip_joint">
                 <state_interface name="position"><param name="initial_value">0.0</param></state_interface>
@@ -151,18 +147,18 @@
             </joint>
             <joint name="${name}_thigh_joint">
-                <state_interface name="position"><param name="initial_value">${t}</param></state_interface>
+                <state_interface name="position"><param name="initial_value">0.0</param></state_interface>
                 <command_interface name="position"/>
                 <state_interface name="velocity"/>
             </joint>
             <joint name="${name}_shin_joint">
-                <state_interface name="position"><param name="initial_value">${s}</param></state_interface>
+                <state_interface name="position"><param name="initial_value">-0.3</param></state_interface>
                 <command_interface name="position"/>
                 <state_interface name="velocity"/>
             </joint>
         </xacro:macro>
-        <xacro:init_pos name="front_left"  t="${init_thigh}" s="${init_shin}"/>
-        <xacro:init_pos name="front_right" t="${init_thigh}" s="${init_shin}"/>
-        <xacro:init_pos name="rear_left"   t="${init_thigh}" s="${init_shin}"/>
-        <xacro:init_pos name="rear_right"  t="${init_thigh}" s="${init_shin}"/>
+        <xacro:init_pos name="front_left"/>
+        <xacro:init_pos name="front_right"/>
+        <xacro:init_pos name="rear_left"/>
+        <xacro:init_pos name="rear_right"/>
     </ros2_control>
     <!-- ==================== GAZEBO PLUGINS ==================== -->
@@ -170,4 +166,5 @@
         <plugin name="gazebo_ros2_control" filename="libgazebo_ros2_control.so">
             <parameters>$(find dog_bringup)/config/controllers.yaml</parameters>
+            <hold_joints>true</hold_joints>
         </plugin>
     </gazebo>

Commit message: wip: STL meshes, gait tuning, xacro pipe fix, initial_value fix
- dog.urdf.xacro: restored ef73995 base, fixed initial_value to match
  physical spawn (thigh=0.0, shin=-0.5), added STL visuals for thigh
  (leg22.STL rpy="0 1.57 0") and shin (leg11.STL rpy="-1.57 0 0"),
  removed non-ASCII comments that broke gazebo_ros2_control rcl parser
- gazebo.launch.py: switched to Python xacro API with .replace('|','')
  to strip autogenerated header that breaks ControllerManager startup,
  added 4s TimerAction delay before trot_node
- controllers.yaml: PID p=80 d=2 on all joints, update_rate=100
- trot_node.cpp: startup ramp from spawn pose (thigh=0, knee=-0.5),
  stationary threshold, smoothed velocity filter
- gait_params.yaml: period=0.8, step_amp_x=0.06, alpha=0.1
- CLAUDE.md: updated to reflect current architecture and known issues
- meshes/: added leg11.STL (shin) and leg22.STL (thigh) from SolidWorks

NOTE: STL mesh alignment and gait stability not yet fully verified.

Co-Authored-By: Claude Sonnet 4.6 <noreply@anthropic.com>

File: src/dog_description/urdf/dog.urdf.xacro (robot description, xacro)
@@ -1,173 +1,137 @@
 <?xml version="1.0"?>
 <robot xmlns:xacro="http://www.ros.org/wiki/xacro" name="dog">
-    <!-- ==================== PROPERTIES ==================== -->
     <xacro:property name="trunk_l" value="0.475"/>
     <xacro:property name="trunk_w" value="0.18"/>
     <xacro:property name="trunk_h" value="0.1"/>
-    <xacro:property name="trunk_m" value="5.0"/>
+    <xacro:property name="trunk_m" value="6.0"/>
     <xacro:property name="hip_l" value="0.06"/>
-    <xacro:property name="hip_m" value="0.15"/>
-    <xacro:property name="hip_r" value="0.02"/>
     <xacro:property name="thigh_l" value="0.144"/>
     <xacro:property name="shin_l" value="0.1525"/>
-    <xacro:property name="thigh_m" value="0.3"/>
-    <xacro:property name="shin_m" value="0.15"/>
+    <xacro:property name="leg_m" value="0.5"/>
     <xacro:property name="leg_r" value="0.02"/>
-    <xacro:property name="foot_r" value="0.02"/>
-    <!-- ==================== MATERIALS ==================== -->
+    <material name="gray"><color rgba="0.5 0.5 0.5 1"/></material>
     <material name="black"><color rgba="0.1 0.1 0.1 1"/></material>
-    <material name="grey"><color rgba="0.6 0.6 0.6 1"/></material>
-    <!-- ==================== INERTIA MACROS ==================== -->
-    <xacro:macro name="box_inertia" params="m l w h">
+    <xacro:macro name="leg_inertia" params="m">
         <inertial>
             <mass value="${m}"/>
-            <inertia ixx="${m/12*(w*w+h*h)}" ixy="0" ixz="0"
-                     iyy="${m/12*(l*l+h*h)}" iyz="0"
-                     izz="${m/12*(l*l+w*w)}"/>
+            <inertia ixx="0.005" ixy="0" ixz="0" iyy="0.005" iyz="0" izz="0.005"/>
         </inertial>
     </xacro:macro>
-    <xacro:macro name="cylinder_inertia_offset" params="m r h ox oy oz">
+    <link name="base_link"><visual><geometry><box size="0.01 0.01 0.01"/></geometry></visual></link>
+    <joint name="base_joint" type="fixed"><parent link="base_link"/><child link="trunk"/></joint>
+    <link name="trunk">
+        <visual><geometry><box size="${trunk_l} ${trunk_w} ${trunk_h}"/></geometry><material name="gray"/></visual>
+        <collision><geometry><box size="${trunk_l} ${trunk_w} ${trunk_h}"/></geometry></collision>
         <inertial>
-            <origin xyz="${ox} ${oy} ${oz}"/>
-            <mass value="${m}"/>
-            <inertia ixx="${m/12*(3*r*r+h*h)}" ixy="0" ixz="0"
-                     iyy="${m/12*(3*r*r+h*h)}" iyz="0"
-                     izz="${m*r*r/2}"/>
+            <mass value="${trunk_m}"/>
+            <origin xyz="-0.05 0 0" rpy="0 0 0"/>
+            <inertia ixx="0.05" ixy="0" ixz="0" iyy="0.1" iyz="0" izz="0.1"/>
         </inertial>
-    </xacro:macro>
-    <!-- ==================== TRUNK ==================== -->
-    <link name="base_link">
-        <visual><geometry><box size="0.01 0.01 0.01"/></geometry></visual>
     </link>
-    <joint name="base_joint" type="fixed">
-        <parent link="base_link"/><child link="trunk"/>
-    </joint>
-    <link name="trunk">
-        <visual>
-            <geometry><box size="${trunk_l} ${trunk_w} ${trunk_h}"/></geometry>
-            <material name="grey"/>
-        </visual>
-        <collision>
-            <geometry><box size="${trunk_l} ${trunk_w} ${trunk_h}"/></geometry>
-        </collision>
-        <xacro:box_inertia m="${trunk_m}" l="${trunk_l}" w="${trunk_w}" h="${trunk_h}"/>
-    </link>
-    <!-- ==================== FOOT FRICTION MACRO ==================== -->
-    <xacro:macro name="foot_friction" params="prefix">
-        <gazebo reference="${prefix}_shin">
-            <mu1>1.5</mu1>
-            <mu2>1.5</mu2>
-            <kp>50000.0</kp>
-            <kd>50.0</kd>
-            <minDepth>0.002</minDepth>
-        </gazebo>
-    </xacro:macro>
-    <!-- ==================== LEG MACRO ==================== -->
     <xacro:macro name="dog_leg" params="prefix side_x side_y">
-        <!-- 1. HIP (Roll) -->
         <joint name="${prefix}_hip_joint" type="revolute">
             <parent link="trunk"/> <child link="${prefix}_hip"/>
             <origin xyz="${side_x * trunk_l/2} ${side_y * trunk_w/2} 0" rpy="0 0 0"/>
             <axis xyz="1 0 0"/>
-            <limit lower="-0.5" upper="0.5" effort="40" velocity="10"/>
-            <dynamics damping="0.5" friction="0.1"/>
+            <limit lower="-0.8" upper="0.8" effort="20" velocity="20"/>
         </joint>
+        <gazebo reference="${prefix}_hip_joint">
+            <implicitSpringDamper>true</implicitSpringDamper>
+        </gazebo>
         <link name="${prefix}_hip">
-            <visual>
-                <origin xyz="0 ${side_y * hip_l/2} 0" rpy="${pi/2} 0 0"/>
-                <geometry><cylinder radius="${hip_r}" length="${hip_l}"/></geometry>
-                <material name="black"/>
-            </visual>
-            <xacro:cylinder_inertia_offset m="${hip_m}" r="${hip_r}" h="${hip_l}"
-                ox="0" oy="${side_y * hip_l/2}" oz="0"/>
+            <visual><geometry><box size="0.05 0.05 0.05"/></geometry><material name="black"/></visual>
+            <xacro:leg_inertia m="0.2"/>
         </link>
-        <!-- 2. THIGH (Pitch) -->
         <joint name="${prefix}_thigh_joint" type="revolute">
             <parent link="${prefix}_hip"/> <child link="${prefix}_thigh"/>
             <origin xyz="0 ${side_y * hip_l} 0" rpy="0 0 0"/>
             <axis xyz="0 1 0"/>
-            <limit lower="-0.5" upper="2.5" effort="40" velocity="10"/>
-            <dynamics damping="0.5" friction="0.1"/>
+            <limit lower="-1.0" upper="4.0" effort="20" velocity="20"/>
         </joint>
+        <gazebo reference="${prefix}_thigh_joint">
+            <implicitSpringDamper>true</implicitSpringDamper>
+        </gazebo>
         <link name="${prefix}_thigh">
             <visual>
-                <origin xyz="0 0 ${-thigh_l/2}"/>
-                <geometry><cylinder radius="${leg_r}" length="${thigh_l}"/></geometry>
-                <material name="grey"/>
+                <origin xyz="0 0 0" rpy="0 1.5707963 0"/>
+                <geometry><mesh filename="package://dog_description/meshes/leg22.STL" scale="0.001 0.001 0.001"/></geometry>
+                <material name="gray"/>
             </visual>
             <collision>
-                <origin xyz="0 0 ${-thigh_l/2}"/>
-                <geometry><cylinder radius="${leg_r}" length="${thigh_l}"/></geometry>
+                <origin xyz="0 0 ${-thigh_l/2}"/><geometry><cylinder radius="${leg_r}" length="${thigh_l - 0.04}"/></geometry>
             </collision>
-            <xacro:cylinder_inertia_offset m="${thigh_m}" r="${leg_r}" h="${thigh_l}"
-                ox="0" oy="0" oz="${-thigh_l/2}"/>
+            <xacro:leg_inertia m="${leg_m}"/>
         </link>
-        <!-- 3. SHIN (Pitch) -->
         <joint name="${prefix}_shin_joint" type="revolute">
             <parent link="${prefix}_thigh"/> <child link="${prefix}_shin"/>
             <origin xyz="0 0 ${-thigh_l}" rpy="0 0 0"/>
             <axis xyz="0 1 0"/>
-            <limit lower="-2.7" upper="-0.3" effort="40" velocity="10"/>
-            <dynamics damping="0.5" friction="0.1"/>
+            <limit lower="-4.0" upper="-0.5" effort="20" velocity="20"/>
         </joint>
+        <gazebo reference="${prefix}_shin_joint">
+            <implicitSpringDamper>true</implicitSpringDamper>
+        </gazebo>
         <link name="${prefix}_shin">
             <visual>
-                <origin xyz="0 0 ${-shin_l/2}"/>
-                <geometry><cylinder radius="${leg_r*0.8}" length="${shin_l}"/></geometry>
+                <origin xyz="0 0 0" rpy="-1.5707963 0 0"/>
+                <geometry><mesh filename="package://dog_description/meshes/leg11.STL" scale="0.001 0.001 0.001"/></geometry>
                 <material name="black"/>
             </visual>
             <collision>
-                <origin xyz="0 0 ${-shin_l/2}"/>
-                <geometry><cylinder radius="${leg_r*0.8}" length="${shin_l}"/></geometry>
+                <origin xyz="0 0 ${-shin_l}"/>
+                <geometry><sphere radius="0.03"/></geometry>
+                <surface>
+                    <friction>
+                        <ode>
+                            <mu>1.0</mu>
+                            <mu2>1.0</mu2>
+                        </ode>
+                    </friction>
+                    <contact>
+                        <ode>
+                            <kp>500000.0</kp>
+                            <kd>100.0</kd>
+                            <minDepth>0.003</minDepth>
+                            <maxVel>0.0</maxVel>
+                        </ode>
+                    </contact>
+                </surface>
             </collision>
-            <!-- Foot sphere -->
-            <collision>
-                <origin xyz="0 0 ${-shin_l}"/>
-                <geometry><sphere radius="${foot_r}"/></geometry>
-            </collision>
-            <xacro:cylinder_inertia_offset m="${shin_m}" r="${leg_r*0.8}" h="${shin_l}"
-                ox="0" oy="0" oz="${-shin_l/2}"/>
+            <xacro:leg_inertia m="${leg_m}"/>
         </link>
-        <xacro:foot_friction prefix="${prefix}"/>
     </xacro:macro>
-    <!-- ==================== INSTANTIATE LEGS ==================== -->
     <xacro:dog_leg prefix="front_left"  side_x="1"  side_y="1"/>
     <xacro:dog_leg prefix="front_right" side_x="1"  side_y="-1"/>
     <xacro:dog_leg prefix="rear_left"   side_x="-1" side_y="1"/>
     <xacro:dog_leg prefix="rear_right"  side_x="-1" side_y="-1"/>
-    <!-- ==================== ROS2 CONTROL ==================== -->
-    <!-- initial_value MUST match the physical spawn pose (thigh=0, shin=-0.3) -->
     <ros2_control name="GazeboSystem" type="system">
         <hardware><plugin>gazebo_ros2_control/GazeboSystem</plugin></hardware>
-        <xacro:macro name="init_pos" params="name">
+        <xacro:macro name="ctrl_joint" params="name thigh_val shin_val">
             <joint name="${name}_hip_joint">
-                <state_interface name="position"><param name="initial_value">0.0</param></state_interface>
                 <command_interface name="position"/>
                 <state_interface name="velocity"/>
+                <state_interface name="position"><param name="initial_value">0.0</param></state_interface>
             </joint>
             <joint name="${name}_thigh_joint">
-                <state_interface name="position"><param name="initial_value">0.0</param></state_interface>
                 <command_interface name="position"/>
                 <state_interface name="velocity"/>
+                <state_interface name="position"><param name="initial_value">${thigh_val}</param></state_interface>
             </joint>
             <joint name="${name}_shin_joint">
-                <state_interface name="position"><param name="initial_value">-0.3</param></state_interface>
                 <command_interface name="position"/>
                 <state_interface name="velocity"/>
+                <state_interface name="position"><param name="initial_value">${shin_val}</param></state_interface>
             </joint>
         </xacro:macro>
-        <xacro:init_pos name="front_left"/>
-        <xacro:init_pos name="front_right"/>
-        <xacro:init_pos name="rear_left"/>
-        <xacro:init_pos name="rear_right"/>
+        <xacro:ctrl_joint name="front_left"  thigh_val="0.0" shin_val="-0.5"/>
+        <xacro:ctrl_joint name="front_right" thigh_val="0.0" shin_val="-0.5"/>
+        <xacro:ctrl_joint name="rear_left"   thigh_val="0.0" shin_val="-0.5"/>
+        <xacro:ctrl_joint name="rear_right"  thigh_val="0.0" shin_val="-0.5"/>
     </ros2_control>
-    <!-- ==================== GAZEBO PLUGINS ==================== -->
     <gazebo>
         <plugin name="gazebo_ros2_control" filename="libgazebo_ros2_control.so">
             <parameters>$(find dog_bringup)/config/controllers.yaml</parameters>
-            <hold_joints>true</hold_joints>
         </plugin>
     </gazebo>
-    <!-- IMU Sensor on trunk -->
     <gazebo reference="trunk">
         <sensor name="imu_sensor" type="imu">
@@ -187,7 +151,5 @@
             </imu>
             <plugin name="imu_plugin" filename="libgazebo_ros_imu_sensor.so">
-                <ros>
-                    <remapping>~/out:=/imu/data</remapping>
-                </ros>
+                <ros><remapping>~/out:=/imu/data</remapping></ros>
                 <initial_orientation_as_reference>false</initial_orientation_as_reference>
                 <frame_name>trunk</frame_name>
