Commit message: fix: gait control overhaul — cmd_vel timeout, gait phase reset, friction & defaults sync
- Add cmd_vel timeout (0.5s) to prevent stuck nonzero velocity from teleop
- Reset gait clock on standing→walking transition (was accumulating during standing → random mid-swing jumps)
- Start gait from double-support phase (gc=0.45) so all legs begin in stance
- Replace model://ground_plane with inline ground plane (mu=100) to guarantee high ground friction
- Remove duplicate <gazebo reference> for shin (was overriding inline surface params)
- Raise foot friction mu 1.0→5.0 in inline collision surface
- Sync all C++ fallback defaults with gait_params.yaml values
- Adjust shin joint upper limit -0.5→-0.1 for nearly vertical spawn pose
- Update URDF initial_value and SPAWN constants to match new limits
- Raise spawn height 0.35→0.42 to prevent ground clipping
- Increase hip joint range ±0.8→±1.0

Co-Authored-By: Claude Opus 4.6 <noreply@anthropic.com>

File: src/dog_description/urdf/dog.urdf.xacro (robot description, xacro)
@@ -34,5 +34,5 @@
             <origin xyz="${side_x * trunk_l/2} ${side_y * trunk_w/2} 0" rpy="0 0 0"/>
             <axis xyz="1 0 0"/>
-            <limit lower="-0.8" upper="0.8" effort="20" velocity="20"/>
+            <limit lower="-1.0" upper="1.0" effort="20" velocity="20"/>
         </joint>
         <gazebo reference="${prefix}_hip_joint">
@@ -67,5 +67,5 @@
             <origin xyz="0 0 ${-thigh_l}" rpy="0 0 0"/>
             <axis xyz="0 1 0"/>
-            <limit lower="-4.0" upper="-0.5" effort="20" velocity="20"/>
+            <limit lower="-4.0" upper="-0.1" effort="20" velocity="20"/>
         </joint>
         <gazebo reference="${prefix}_shin_joint">
@@ -83,5 +83,5 @@
                 <surface>
                     <friction>
-                        <ode><mu>1.0</mu><mu2>1.0</mu2></ode>
+                        <ode><mu>5.0</mu><mu2>5.0</mu2></ode>
                     </friction>
                     <contact>
@@ -97,12 +97,4 @@
             <xacro:leg_inertia m="${leg_m}"/>
         </link>
-        <gazebo reference="${prefix}_shin">
-            <mu1>1.0</mu1>
-            <mu2>1.0</mu2>
-            <kp>500000</kp>
-            <kd>100</kd>
-            <minDepth>0.003</minDepth>
-            <maxVel>0</maxVel>
-        </gazebo>
     </xacro:macro>
     <xacro:dog_leg prefix="front_left"  side_x="1"  side_y="1"/>
@@ -129,8 +121,8 @@
             </joint>
         </xacro:macro>
-        <xacro:ctrl_joint name="front_left"  thigh_val="0.0" shin_val="-0.5"/>
-        <xacro:ctrl_joint name="front_right" thigh_val="0.0" shin_val="-0.5"/>
-        <xacro:ctrl_joint name="rear_left"   thigh_val="0.0" shin_val="-0.5"/>
-        <xacro:ctrl_joint name="rear_right"  thigh_val="0.0" shin_val="-0.5"/>
+        <xacro:ctrl_joint name="front_left"  thigh_val="0.0" shin_val="-0.1"/>
+        <xacro:ctrl_joint name="front_right" thigh_val="0.0" shin_val="-0.1"/>
+        <xacro:ctrl_joint name="rear_left"   thigh_val="0.0" shin_val="-0.1"/>
+        <xacro:ctrl_joint name="rear_right"  thigh_val="0.0" shin_val="-0.1"/>
     </ros2_control>
     <gazebo>
