Commit message: fix: remove cyrillic from urdf and add pid gains

File: src/dog_description/urdf/dog.urdf.xacro (robot description, xacro)
@@ -1,191 +1,196 @@
 <?xml version="1.0"?>
-<robot xmlns:xacro="http://ros.org/wiki/xacro" name="dog">
-  <!-- ===== параметры ===== -->
-  <xacro:property name="body_length" value="0.475"/>
-  <xacro:property name="body_width"  value="0.18"/>
-  <xacro:property name="body_height" value="0.10"/>
-  <xacro:property name="thigh_length" value="0.144"/>
-  <xacro:property name="shin_length" value="0.1525"/>
-  <xacro:property name="leg_radius" value="0.02"/>
-  <xacro:property name="leg_mass" value="0.2"/>
-  <!-- ===== base_link ===== -->
-  <link name="base_link">
-    <visual>
-      <origin xyz="0 0 0" rpy="0 0 0"/>
-      <geometry>
-        <box size="${body_length} ${body_width} ${body_height}"/>
-      </geometry>
-      <material name="gray"><color rgba="0.5 0.5 0.5 1"/></material>
-    </visual>
-    <collision>
-      <origin xyz="0 0 0" rpy="0 0 0"/>
-      <geometry>
-        <box size="${body_length} ${body_width} ${body_height}"/>
-      </geometry>
-    </collision>
-    <inertial>
-      <mass value="5.0"/>
-      <inertia ixx="0.1" ixy="0" ixz="0" iyy="0.1" iyz="0" izz="0.1"/>
-    </inertial>
-  </link>
-  <!-- ===== макрос лапы (hip-thigh-shin) ===== -->
-  <xacro:macro name="leg" params="name x y">
-    <!-- hip -->
-    <link name="${name}_hip">
-      <visual>
+<robot xmlns:xacro="http://www.ros.org/wiki/xacro" name="dog">
+    <!-- ================================================================== -->
+    <!--                           CONSTANTS & MACROS                       -->
+    <!-- ================================================================== -->
+    <xacro:property name="trunk_l" value="0.5"/>
+    <xacro:property name="trunk_w" value="0.3"/>
+    <xacro:property name="trunk_h" value="0.15"/>
+    <xacro:property name="trunk_m" value="10.0"/>
+    <xacro:property name="hip_l" value="0.05"/>
+    <xacro:property name="thigh_l" value="0.25"/>
+    <xacro:property name="shin_l" value="0.25"/>
+    <xacro:property name="leg_m" value="1.0"/>
+    <xacro:property name="leg_r" value="0.03"/>
+    <xacro:macro name="box_inertia" params="m x y z">
+        <inertial>
+            <mass value="${m}"/>
+            <inertia ixx="${m/12 * (y*y + z*z)}" ixy="0" ixz="0"
+                     iyy="${m/12 * (x*x + z*z)}" iyz="0"
+                     izz="${m/12 * (x*x + y*y)}"/>
+        </inertial>
+    </xacro:macro>
+    <xacro:macro name="cylinder_inertia" params="m r h">
+        <inertial>
+            <mass value="${m}"/>
+            <inertia ixx="${m/12 * (3*r*r + h*h)}" ixy="0" ixz="0"
+                     iyy="${m/12 * (3*r*r + h*h)}" iyz="0"
+                     izz="${m/2 * (r*r)}"/>
+        </inertial>
+    </xacro:macro>
+    <material name="gray"><color rgba="0.5 0.5 0.5 1"/></material>
+    <material name="black"><color rgba="0.1 0.1 0.1 1"/></material>
+    <!-- ================================================================== -->
+    <!--                           ROBOT DESCRIPTION                        -->
+    <!-- ================================================================== -->
+    <!-- 1. BASE_LINK (VIRTUAL) -->
+    <link name="base_link">
+        <visual>
+            <geometry><box size="0.01 0.01 0.01"/></geometry>
+            <material name="gray"/>
+        </visual>
+    </link>
+    <!-- 2. TRUNK (BODY) -->
+    <joint name="base_joint" type="fixed">
+        <parent link="base_link"/>
+        <child link="trunk"/>
         <origin xyz="0 0 0" rpy="0 0 0"/>
-        <geometry>
-          <cylinder radius="${leg_radius}" length="0.05"/>
-        </geometry>
-        <material name="black"><color rgba="0 0 0 1"/></material>
-      </visual>
-      <collision>
-        <origin xyz="0 0 0" rpy="0 0 0"/>
-        <geometry>
-          <cylinder radius="${leg_radius}" length="0.05"/>
-        </geometry>
-      </collision>
-      <inertial>
-        <mass value="${leg_mass}"/>
-        <inertia ixx="0.001" ixy="0" ixz="0" iyy="0.001" iyz="0" izz="0.001"/>
-      </inertial>
+    </joint>
+    <link name="trunk">
+        <visual>
+            <geometry><box size="${trunk_l} ${trunk_w} ${trunk_h}"/></geometry>
+            <material name="gray"/>
+        </visual>
+        <collision>
+            <geometry><box size="${trunk_l} ${trunk_w} ${trunk_h}"/></geometry>
+        </collision>
+        <xacro:box_inertia m="${trunk_m}" x="${trunk_l}" y="${trunk_w}" z="${trunk_h}"/>
     </link>
-    <joint name="${name}_hip_joint" type="revolute">
-      <parent link="base_link"/>
-      <child  link="${name}_hip"/>
-      <origin xyz="${x} ${y} 0" rpy="0 0 0"/>
-      <axis xyz="0 0 1"/>
-      <limit lower="-1.57" upper="1.57" effort="10" velocity="1"/>
-    </joint>
-    <!-- thigh -->
-    <link name="${name}_thigh">
-      <visual>
-        <origin xyz="0 0 -${thigh_length/2.0}" rpy="0 0 0"/>
-        <geometry>
-          <cylinder radius="${leg_radius}" length="${thigh_length}"/>
-        </geometry>
-        <material name="blue"><color rgba="0 0 1 1"/></material>
-      </visual>
-      <collision>
-        <origin xyz="0 0 -${thigh_length/2.0}" rpy="0 0 0"/>
-        <geometry>
-          <cylinder radius="${leg_radius}" length="${thigh_length}"/>
-        </geometry>
-      </collision>
-      <inertial>
-        <mass value="${leg_mass}"/>
-        <inertia ixx="0.001" ixy="0" ixz="0" iyy="0.001" iyz="0" izz="0.001"/>
-      </inertial>
-    </link>
-    <joint name="${name}_thigh_joint" type="revolute">
-      <parent link="${name}_hip"/>
-      <child  link="${name}_thigh"/>
-      <origin xyz="0 0 0" rpy="0 0 0"/>
-      <axis xyz="1 0 0"/>
-      <limit lower="-1.57" upper="1.57" effort="10" velocity="1"/>
-    </joint>
-    <!-- shin -->
-    <link name="${name}_shin">
-      <visual>
-        <origin xyz="0 0 -${shin_length/2.0}" rpy="0 0 0"/>
-        <geometry>
-          <cylinder radius="${leg_radius}" length="${shin_length}"/>
-        </geometry>
-        <material name="red"><color rgba="1 0 0 1"/></material>
-      </visual>
-      <collision>
-        <origin xyz="0 0 -${shin_length/2.0}" rpy="0 0 0"/>
-        <geometry>
-          <cylinder radius="${leg_radius}" length="${shin_length}"/>
-        </geometry>
-      </collision>
-      <inertial>
-        <mass value="${leg_mass}"/>
-        <inertia ixx="0.001" ixy="0" ixz="0" iyy="0.001" iyz="0" izz="0.001"/>
-      </inertial>
-    </link>
-    <joint name="${name}_shin_joint" type="revolute">
-      <parent link="${name}_thigh"/>
-      <child  link="${name}_shin"/>
-      <origin xyz="0 0 -${thigh_length}" rpy="0 0 0"/>
-      <axis xyz="1 0 0"/>
-      <limit lower="-1.57" upper="1.57" effort="10" velocity="1"/>
-    </joint>
-  </xacro:macro>
-  <!-- ===== четыре лапы ===== -->
-  <xacro:leg name="front_left"  x="${body_length/2.0}"  y="${body_width/2.0}"/>
-  <xacro:leg name="front_right" x="${body_length/2.0}"  y="-${body_width/2.0}"/>
-  <xacro:leg name="rear_left"   x="-${body_length/2.0}" y="${body_width/2.0}"/>
-  <xacro:leg name="rear_right"  x="-${body_length/2.0}" y="-${body_width/2.0}"/>
-  <!-- ===== ros2_control ===== -->
-  <ros2_control name="DogSystem" type="system">
-    <hardware>
-      <plugin>gazebo_ros2_control/GazeboSystem</plugin>
-    </hardware>
-    <!-- перечисляем все суставы -->
-    <joint name="front_left_hip_joint">
-      <command_interface name="position"/>
-      <state_interface name="position"/>
-      <state_interface name="velocity"/>
-    </joint>
-    <joint name="front_left_thigh_joint">
-      <command_interface name="position"/>
-      <state_interface name="position"/>
-      <state_interface name="velocity"/>
-    </joint>
-    <joint name="front_left_shin_joint">
-      <command_interface name="position"/>
-      <state_interface name="position"/>
-      <state_interface name="velocity"/>
-    </joint>
-    <joint name="front_right_hip_joint">
-      <command_interface name="position"/>
-      <state_interface name="position"/>
-      <state_interface name="velocity"/>
-    </joint>
-    <joint name="front_right_thigh_joint">
-      <command_interface name="position"/>
-      <state_interface name="position"/>
-      <state_interface name="velocity"/>
-    </joint>
-    <joint name="front_right_shin_joint">
-      <command_interface name="position"/>
-      <state_interface name="position"/>
-      <state_interface name="velocity"/>
-    </joint>
-    <joint name="rear_left_hip_joint">
-      <command_interface name="position"/>
-      <state_interface name="position"/>
-      <state_interface name="velocity"/>
-    </joint>
-    <joint name="rear_left_thigh_joint">
-      <command_interface name="position"/>
-      <state_interface name="position"/>
-      <state_interface name="velocity"/>
-    </joint>
-    <joint name="rear_left_shin_joint">
-      <command_interface name="position"/>
-      <state_interface name="position"/>
-      <state_interface name="velocity"/>
-    </joint>
-    <joint name="rear_right_hip_joint">
-      <command_interface name="position"/>
-      <state_interface name="position"/>
-      <state_interface name="velocity"/>
-    </joint>
-    <joint name="rear_right_thigh_joint">
-      <command_interface name="position"/>
-      <state_interface name="position"/>
-      <state_interface name="velocity"/>
-    </joint>
-    <joint name="rear_right_shin_joint">
-      <command_interface name="position"/>
-      <state_interface name="position"/>
-      <state_interface name="velocity"/>
-    </joint>
-  </ros2_control>
-  <!-- ===== Gazebo плагин ===== -->
-  <gazebo reference="base_link">
-    <plugin name="gazebo_ros2_control" filename="libgazebo_ros2_control.so"/>
-  </gazebo>
+    <!-- 3. LEG MACRO -->
+    <xacro:macro name="dog_leg" params="prefix side_x side_y">
+        <!-- === HIP JOINT (Abduction/Adduction - Roll) === -->
+        <joint name="${prefix}_hip_joint" type="revolute">
+            <parent link="trunk"/>
+            <child link="${prefix}_hip"/>
+            <origin xyz="${side_x * trunk_l/2} ${side_y * trunk_w/2} 0" rpy="0 0 0"/>
+            <axis xyz="1 0 0"/>
+            <limit lower="-0.7" upper="0.7" effort="100" velocity="10"/>
+            <dynamics damping="0.5" friction="0.1"/>
+        </joint>
+        <link name="${prefix}_hip">
+            <visual>
+                <origin xyz="0 ${side_y * 0.05} 0"/>
+                <geometry><box size="0.1 0.1 0.1"/></geometry>
+                <material name="black"/>
+            </visual>
+            <collision>
+                <origin xyz="0 ${side_y * 0.05} 0"/>
+                <geometry><box size="0.1 0.1 0.1"/></geometry>
+            </collision>
+            <xacro:box_inertia m="0.5" x="0.1" y="0.1" z="0.1"/>
+        </link>
+        <!-- === THIGH JOINT (Flexion/Extension - Pitch) === -->
+        <joint name="${prefix}_thigh_joint" type="revolute">
+            <parent link="${prefix}_hip"/>
+            <child link="${prefix}_thigh"/>
+            <origin xyz="0 ${side_y * 0.05} 0" rpy="0 0 0"/>
+            <axis xyz="0 1 0"/>
+            <limit lower="-1.5" upper="1.5" effort="100" velocity="10"/>
+            <dynamics damping="0.5" friction="0.1"/>
+        </joint>
+        <link name="${prefix}_thigh">
+            <visual>
+                <origin xyz="0 0 ${-thigh_l/2}" rpy="0 0 0"/>
+                <geometry><cylinder radius="${leg_r}" length="${thigh_l}"/></geometry>
+                <material name="gray"/>
+            </visual>
+            <collision>
+                <origin xyz="0 0 ${-thigh_l/2}" rpy="0 0 0"/>
+                <geometry><cylinder radius="${leg_r}" length="${thigh_l}"/></geometry>
+            </collision>
+            <xacro:cylinder_inertia m="${leg_m}" r="${leg_r}" h="${thigh_l}"/>
+        </link>
+        <!-- === SHIN JOINT (Knee - Pitch) === -->
+        <joint name="${prefix}_shin_joint" type="revolute">
+            <parent link="${prefix}_thigh"/>
+            <child link="${prefix}_shin"/>
+            <origin xyz="0 0 ${-thigh_l}" rpy="0 0 0"/>
+            <axis xyz="0 1 0"/>
+            <limit lower="-2.5" upper="0.0" effort="100" velocity="10"/>
+            <dynamics damping="0.5" friction="0.1"/>
+        </joint>
+        <link name="${prefix}_shin">
+            <visual>
+                <origin xyz="0 0 ${-shin_l/2}" rpy="0 0 0"/>
+                <geometry><cylinder radius="${leg_r*0.8}" length="${shin_l}"/></geometry>
+                <material name="black"/>
+            </visual>
+            <collision>
+                <origin xyz="0 0 ${-shin_l/2}" rpy="0 0 0"/>
+                <geometry><cylinder radius="${leg_r*0.8}" length="${shin_l}"/></geometry>
+                <surface>
+                    <friction>
+                        <ode>
+                            <mu>1.0</mu>
+                            <mu2>1.0</mu2>
+                        </ode>
+                    </friction>
+                </surface>
+            </collision>
+            <xacro:cylinder_inertia m="${leg_m}" r="${leg_r*0.8}" h="${shin_l}"/>
+        </link>
+    </xacro:macro>
+    <!-- 4. GENERATE LEGS -->
+    <xacro:dog_leg prefix="front_left"  side_x="1"  side_y="1"/>
+    <xacro:dog_leg prefix="front_right" side_x="1"  side_y="-1"/>
+    <xacro:dog_leg prefix="rear_left"   side_x="-1" side_y="1"/>
+    <xacro:dog_leg prefix="rear_right"  side_x="-1" side_y="-1"/>
+    <!-- ================================================================== -->
+    <!--                          ROS2 CONTROL SETUP                        -->
+    <!-- ================================================================== -->
+    <ros2_control name="GazeboSystem" type="system">
+        <hardware>
+            <plugin>gazebo_ros2_control/GazeboSystem</plugin>
+        </hardware>
+        <!-- FRONT LEFT -->
+        <joint name="front_left_hip_joint">
+            <command_interface name="position"/><state_interface name="position"/><state_interface name="velocity"/>
+        </joint>
+        <joint name="front_left_thigh_joint">
+            <command_interface name="position"/><state_interface name="position"/><state_interface name="velocity"/>
+        </joint>
+        <joint name="front_left_shin_joint">
+            <command_interface name="position"/><state_interface name="position"/><state_interface name="velocity"/>
+        </joint>
+        <!-- FRONT RIGHT -->
+        <joint name="front_right_hip_joint">
+            <command_interface name="position"/><state_interface name="position"/><state_interface name="velocity"/>
+        </joint>
+        <joint name="front_right_thigh_joint">
+            <command_interface name="position"/><state_interface name="position"/><state_interface name="velocity"/>
+        </joint>
+        <joint name="front_right_shin_joint">
+            <command_interface name="position"/><state_interface name="position"/><state_interface name="velocity"/>
+        </joint>
+        <!-- REAR LEFT -->
+        <joint name="rear_left_hip_joint">
+            <command_interface name="position"/><state_interface name="position"/><state_interface name="velocity"/>
+        </joint>
+        <joint name="rear_left_thigh_joint">
+            <command_interface name="position"/><state_interface name="position"/><state_interface name="velocity"/>
+        </joint>
+        <joint name="rear_left_shin_joint">
+            <command_interface name="position"/><state_interface name="position"/><state_interface name="velocity"/>
+        </joint>
+        <!-- REAR RIGHT -->
+        <joint name="rear_right_hip_joint">
+            <command_interface name="position"/><state_interface name="position"/><state_interface name="velocity"/>
+        </joint>
+        <joint name="rear_right_thigh_joint">
+            <command_interface name="position"/><state_interface name="position"/><state_interface name="velocity"/>
+        </joint>
+        <joint name="rear_right_shin_joint">
+            <command_interface name="position"/><state_interface name="position"/><state_interface name="velocity"/>
+        </joint>
+    </ros2_control>
+    <!-- ================================================================== -->
+    <!--                           GAZEBO PLUGIN                            -->
+    <!-- ================================================================== -->
+    <gazebo>
+         <plugin name="gazebo_ros2_control" filename="libgazebo_ros2_control.so">
+            <parameters>$(find dog_controllers)/config/controllers.yaml</parameters>
+            <robot_param>robot_description</robot_param>
+            <robot_param_node>robot_state_publisher</robot_param_node>
+        </plugin>
+    </gazebo>
 </robot>
