Commit message: рабочая физика, робот стоит и почти готов к написанию движения, скользит в симуляции

File: src/dog_description/urdf/dog.urdf.xacro (robot description, xacro)
@@ -1,22 +1,17 @@
 <?xml version="1.0"?>
 <robot xmlns:xacro="http://www.ros.org/wiki/xacro" name="dog">
-    <!-- ================================================================== -->
-    <!--                           CONSTANTS & MACROS                       -->
-    <!-- ================================================================== -->
     <xacro:property name="trunk_l" value="0.5"/>
     <xacro:property name="trunk_w" value="0.3"/>
     <xacro:property name="trunk_h" value="0.15"/>
-    <xacro:property name="trunk_m" value="10.0"/>
+    <xacro:property name="trunk_m" value="5.0"/>
     <xacro:property name="hip_l" value="0.05"/>
     <xacro:property name="thigh_l" value="0.25"/>
     <xacro:property name="shin_l" value="0.25"/>
-    <xacro:property name="leg_m" value="1.0"/>
+    <xacro:property name="leg_m" value="2.0"/>
     <xacro:property name="leg_r" value="0.03"/>
     <xacro:macro name="box_inertia" params="m x y z">
         <inertial>
             <mass value="${m}"/>
-            <inertia ixx="${m/12 * (y*y + z*z)}" ixy="0" ixz="0"
-                     iyy="${m/12 * (x*x + z*z)}" iyz="0"
-                     izz="${m/12 * (x*x + y*y)}"/>
+            <inertia ixx="0.1" ixy="0" ixz="0" iyy="0.1" iyz="0" izz="0.1"/>
         </inertial>
     </xacro:macro>
@@ -24,26 +19,14 @@
         <inertial>
             <mass value="${m}"/>
-            <inertia ixx="${m/12 * (3*r*r + h*h)}" ixy="0" ixz="0"
-                     iyy="${m/12 * (3*r*r + h*h)}" iyz="0"
-                     izz="${m/2 * (r*r)}"/>
+            <inertia ixx="0.01" ixy="0" ixz="0" iyy="0.1" iyz="0" izz="0.1"/>
         </inertial>
     </xacro:macro>
     <material name="gray"><color rgba="0.5 0.5 0.5 1"/></material>
     <material name="black"><color rgba="0.1 0.1 0.1 1"/></material>
-    <!-- ================================================================== -->
-    <!--                           ROBOT DESCRIPTION                        -->
-    <!-- ================================================================== -->
-    <!-- 1. BASE_LINK (VIRTUAL) -->
-    <link name="base_link">
-        <visual>
-            <geometry><box size="0.01 0.01 0.01"/></geometry>
-            <material name="gray"/>
-        </visual>
-    </link>
-    <!-- 2. TRUNK (BODY) -->
+    <!-- BASE & TRUNK -->
+    <link name="base_link"><visual><geometry><box size="0.01 0.01 0.01"/></geometry></visual></link>
     <joint name="base_joint" type="fixed">
         <parent link="base_link"/>
         <child link="trunk"/>
-        <origin xyz="0 0 0" rpy="0 0 0"/>
     </joint>
     <link name="trunk">
@@ -57,7 +40,7 @@
         <xacro:box_inertia m="${trunk_m}" x="${trunk_l}" y="${trunk_w}" z="${trunk_h}"/>
     </link>
-    <!-- 3. LEG MACRO -->
+    <!-- LEG MACRO -->
     <xacro:macro name="dog_leg" params="prefix side_x side_y">
-        <!-- === HIP JOINT (Abduction/Adduction - Roll) === -->
+        <!-- HIP -->
         <joint name="${prefix}_hip_joint" type="revolute">
             <parent link="trunk"/>
@@ -65,6 +48,6 @@
             <origin xyz="${side_x * trunk_l/2} ${side_y * trunk_w/2} 0" rpy="0 0 0"/>
             <axis xyz="1 0 0"/>
-            <limit lower="-0.7" upper="0.7" effort="100" velocity="10"/>
-            <dynamics damping="0.5" friction="0.1"/>
+            <limit lower="-0.7" upper="0.7" effort="50" velocity="5"/>
+            <dynamics damping="1.0" friction="0.5"/>
         </joint>
         <link name="${prefix}_hip">
@@ -74,11 +57,8 @@
                 <material name="black"/>
             </visual>
-            <collision>
-                <origin xyz="0 ${side_y * 0.05} 0"/>
-                <geometry><box size="0.1 0.1 0.1"/></geometry>
-            </collision>
+            <!-- <collision> ... </collision> -->
             <xacro:box_inertia m="0.5" x="0.1" y="0.1" z="0.1"/>
         </link>
-        <!-- === THIGH JOINT (Flexion/Extension - Pitch) === -->
+        <!-- THIGH -->
         <joint name="${prefix}_thigh_joint" type="revolute">
             <parent link="${prefix}_hip"/>
@@ -86,6 +66,6 @@
             <origin xyz="0 ${side_y * 0.05} 0" rpy="0 0 0"/>
             <axis xyz="0 1 0"/>
-            <limit lower="-1.5" upper="1.5" effort="100" velocity="10"/>
-            <dynamics damping="0.5" friction="0.1"/>
+            <limit lower="-1.5" upper="1.5" effort="50" velocity="5"/>
+            <dynamics damping="1.0" friction="0.5"/>
         </joint>
         <link name="${prefix}_thigh">
@@ -97,9 +77,9 @@
             <collision>
                 <origin xyz="0 0 ${-thigh_l/2}" rpy="0 0 0"/>
-                <geometry><cylinder radius="${leg_r}" length="${thigh_l}"/></geometry>
+                <geometry><cylinder radius="0.02" length="${thigh_l - 0.1}"/></geometry>
             </collision>
             <xacro:cylinder_inertia m="${leg_m}" r="${leg_r}" h="${thigh_l}"/>
         </link>
-        <!-- === SHIN JOINT (Knee - Pitch) === -->
+        <!-- SHIN -->
         <joint name="${prefix}_shin_joint" type="revolute">
             <parent link="${prefix}_thigh"/>
@@ -107,6 +87,6 @@
             <origin xyz="0 0 ${-thigh_l}" rpy="0 0 0"/>
             <axis xyz="0 1 0"/>
-            <limit lower="-2.5" upper="0.0" effort="100" velocity="10"/>
-            <dynamics damping="0.5" friction="0.1"/>
+            <limit lower="-2.5" upper="0.0" effort="50" velocity="5"/>
+            <dynamics damping="1.0" friction="0.5"/>
         </joint>
         <link name="${prefix}_shin">
@@ -117,13 +97,13 @@
             </visual>
             <collision>
-                <origin xyz="0 0 ${-shin_l/2}" rpy="0 0 0"/>
-                <geometry><cylinder radius="${leg_r*0.8}" length="${shin_l}"/></geometry>
+                <origin xyz="0 0 ${-shin_l}" rpy="0 0 0"/>
+                <geometry><sphere radius="0.04"/></geometry>
                 <surface>
                     <friction>
-                        <ode>
-                            <mu>1.0</mu>
-                            <mu2>1.0</mu2>
-                        </ode>
+                        <ode><mu>200.0</mu><mu2>200.0</mu2></ode>
                     </friction>
+                    <contact>
+                        <ode><kp>100000.0</kp><kd>1000.0</kd><min_depth>0.001</min_depth></ode>
+                    </contact>
                 </surface>
             </collision>
@@ -131,66 +111,42 @@
         </link>
     </xacro:macro>
-    <!-- 4. GENERATE LEGS -->
     <xacro:dog_leg prefix="front_left"  side_x="1"  side_y="1"/>
     <xacro:dog_leg prefix="front_right" side_x="1"  side_y="-1"/>
     <xacro:dog_leg prefix="rear_left"   side_x="-1" side_y="1"/>
     <xacro:dog_leg prefix="rear_right"  side_x="-1" side_y="-1"/>
-    <!-- ================================================================== -->
-    <!--                          ROS2 CONTROL SETUP                        -->
-    <!-- ================================================================== -->
     <ros2_control name="GazeboSystem" type="system">
-        <hardware>
-            <plugin>gazebo_ros2_control/GazeboSystem</plugin>
-        </hardware>
-        <!-- FRONT LEFT -->
-        <joint name="front_left_hip_joint">
-            <command_interface name="position"/><state_interface name="position"/><state_interface name="velocity"/>
-        </joint>
-        <joint name="front_left_thigh_joint">
-            <command_interface name="position"/><state_interface name="position"/><state_interface name="velocity"/>
-        </joint>
-        <joint name="front_left_shin_joint">
-            <command_interface name="position"/><state_interface name="position"/><state_interface name="velocity"/>
-        </joint>
-        <!-- FRONT RIGHT -->
-        <joint name="front_right_hip_joint">
-            <command_interface name="position"/><state_interface name="position"/><state_interface name="velocity"/>
-        </joint>
-        <joint name="front_right_thigh_joint">
-            <command_interface name="position"/><state_interface name="position"/><state_interface name="velocity"/>
-        </joint>
-        <joint name="front_right_shin_joint">
-            <command_interface name="position"/><state_interface name="position"/><state_interface name="velocity"/>
-        </joint>
-        <!-- REAR LEFT -->
-        <joint name="rear_left_hip_joint">
-            <command_interface name="position"/><state_interface name="position"/><state_interface name="velocity"/>
-        </joint>
-        <joint name="rear_left_thigh_joint">
-            <command_interface name="position"/><state_interface name="position"/><state_interface name="velocity"/>
-        </joint>
-        <joint name="rear_left_shin_joint">
-            <command_interface name="position"/><state_interface name="position"/><state_interface name="velocity"/>
-        </joint>
-        <!-- REAR RIGHT -->
-        <joint name="rear_right_hip_joint">
-            <command_interface name="position"/><state_interface name="position"/><state_interface name="velocity"/>
-        </joint>
-        <joint name="rear_right_thigh_joint">
-            <command_interface name="position"/><state_interface name="position"/><state_interface name="velocity"/>
-        </joint>
-        <joint name="rear_right_shin_joint">
-            <command_interface name="position"/><state_interface name="position"/><state_interface name="velocity"/>
-        </joint>
+        <hardware><plugin>gazebo_ros2_control/GazeboSystem</plugin></hardware>
+        <joint name="front_left_hip_joint"><command_interface name="position"/><state_interface name="velocity"/><state_interface name="position"><param name="initial_value">0.0</param></state_interface></joint>
+        <joint name="front_left_thigh_joint"><command_interface name="position"/><state_interface name="velocity"/><state_interface name="position"><param name="initial_value">0.9</param></state_interface></joint>
+        <joint name="front_left_shin_joint"><command_interface name="position"/><state_interface name="velocity"/><state_interface name="position"><param name="initial_value">-1.8</param></state_interface></joint>
+        <joint name="front_right_hip_joint"><command_interface name="position"/><state_interface name="velocity"/><state_interface name="position"><param name="initial_value">0.0</param></state_interface></joint>
+        <joint name="front_right_thigh_joint"><command_interface name="position"/><state_interface name="velocity"/><state_interface name="position"><param name="initial_value">0.9</param></state_interface></joint>
+        <joint name="front_right_shin_joint"><command_interface name="position"/><state_interface name="velocity"/><state_interface name="position"><param name="initial_value">-1.8</param></state_interface></joint>
+        <joint name="rear_left_hip_joint"><command_interface name="position"/><state_interface name="velocity"/><state_interface name="position"><param name="initial_value">0.0</param></state_interface></joint>
+        <joint name="rear_left_thigh_joint"><command_interface name="position"/><state_interface name="velocity"/><state_interface name="position"><param name="initial_value">0.9</param></state_interface></joint>
+        <joint name="rear_left_shin_joint"><command_interface name="position"/><state_interface name="velocity"/><state_interface name="position"><param name="initial_value">-1.8</param></state_interface></joint>
+        <joint name="rear_right_hip_joint"><command_interface name="position"/><state_interface name="velocity"/><state_interface name="position"><param name="initial_value">0.0</param></state_interface></joint>
+        <joint name="rear_right_thigh_joint"><command_interface name="position"/><state_interface name="velocity"/><state_interface name="position"><param name="initial_value">0.9</param></state_interface></joint>
+        <joint name="rear_right_shin_joint"><command_interface name="position"/><state_interface name="velocity"/><state_interface name="position"><param name="initial_value">-1.8</param></state_interface></joint>
     </ros2_control>
-    <!-- ================================================================== -->
-    <!--                           GAZEBO PLUGIN                            -->
-    <!-- ================================================================== -->
     <gazebo>
-         <plugin name="gazebo_ros2_control" filename="libgazebo_ros2_control.so">
+        <plugin name="gazebo_ros2_control" filename="libgazebo_ros2_control.so">
             <parameters>$(find dog_controllers)/config/controllers.yaml</parameters>
-            <robot_param>robot_description</robot_param>
-            <robot_param_node>robot_state_publisher</robot_param_node>
         </plugin>
     </gazebo>
+    <xacro:macro name="foot_physics" params="prefix">
+        <gazebo reference="${prefix}_shin">
+            <mu1>10.0</mu1>
+            <mu2>10.0</mu2>
+            <kp>1000000.0</kp>
+            <kd>1.0</kd>
+            <maxVel>0.0</maxVel>
+            <minDepth>0.002</minDepth>
+            <material>Gazebo/Black</material>
+        </gazebo>
+    </xacro:macro>
+    <xacro:foot_physics prefix="front_left"/>
+    <xacro:foot_physics prefix="front_right"/>
+    <xacro:foot_physics prefix="rear_left"/>
+    <xacro:foot_physics prefix="rear_right"/>
 </robot>

Commit message: реальные размеры, начало генерации походки, чуть скользит

File: src/dog_description/urdf/dog.urdf.xacro (robot description, xacro)
@@ -1,13 +1,13 @@
 <?xml version="1.0"?>
 <robot xmlns:xacro="http://www.ros.org/wiki/xacro" name="dog">
-    <xacro:property name="trunk_l" value="0.5"/>
-    <xacro:property name="trunk_w" value="0.3"/>
-    <xacro:property name="trunk_h" value="0.15"/>
-    <xacro:property name="trunk_m" value="5.0"/>
-    <xacro:property name="hip_l" value="0.05"/>
-    <xacro:property name="thigh_l" value="0.25"/>
-    <xacro:property name="shin_l" value="0.25"/>
-    <xacro:property name="leg_m" value="2.0"/>
-    <xacro:property name="leg_r" value="0.03"/>
+    <xacro:property name="trunk_l" value="0.47543"/> <!-- 475.43  -->
+    <xacro:property name="trunk_w" value="0.1807"/>  <!-- 180.7 -->
+    <xacro:property name="trunk_h" value="0.1"/>     <!-- -->
+    <xacro:property name="trunk_m" value="6.0"/>     <!--  -->
+    <xacro:property name="hip_l" value="0.06"/>      <!-- -->
+    <xacro:property name="thigh_l" value="0.144"/>   <!-- 144 -->
+    <xacro:property name="shin_l" value="0.1525"/>   <!-- 152.5  -->
+    <xacro:property name="leg_m" value="0.5"/>       <!-- 0.5  -->
+    <xacro:property name="leg_r" value="0.02"/>      <!--  -->
     <xacro:macro name="box_inertia" params="m x y z">
         <inertial>
@@ -77,5 +77,5 @@
             <collision>
                 <origin xyz="0 0 ${-thigh_l/2}" rpy="0 0 0"/>
-                <geometry><cylinder radius="0.02" length="${thigh_l - 0.1}"/></geometry>
+                <geometry><cylinder radius="0.015" length="${thigh_l - 0.04}"/></geometry>
             </collision>
             <xacro:cylinder_inertia m="${leg_m}" r="${leg_r}" h="${thigh_l}"/>
