Commit message: ниче не изменилось, переписанный urdf и trot, все еще нерабочее

File: src/dog_description/urdf/dog.urdf.xacro (robot description, xacro)
@@ -1,17 +1,19 @@
 <?xml version="1.0"?>
 <robot xmlns:xacro="http://www.ros.org/wiki/xacro" name="dog">
-    <xacro:property name="trunk_l" value="0.47543"/> <!-- 475.43  -->
-    <xacro:property name="trunk_w" value="0.1807"/>  <!-- 180.7 -->
-    <xacro:property name="trunk_h" value="0.1"/>     <!-- -->
-    <xacro:property name="trunk_m" value="6.0"/>     <!--  -->
-    <xacro:property name="hip_l" value="0.06"/>      <!-- -->
-    <xacro:property name="thigh_l" value="0.144"/>   <!-- 144 -->
-    <xacro:property name="shin_l" value="0.1525"/>   <!-- 152.5  -->
-    <xacro:property name="leg_m" value="0.5"/>       <!-- 0.5  -->
-    <xacro:property name="leg_r" value="0.02"/>      <!--  -->
+    <xacro:property name="trunk_l" value="0.475"/>
+    <xacro:property name="trunk_w" value="0.18"/>
+    <xacro:property name="trunk_h" value="0.1"/>
+    <xacro:property name="trunk_m" value="6.0"/>
+    <xacro:property name="hip_l" value="0.06"/>
+    <xacro:property name="thigh_l" value="0.144"/>
+    <xacro:property name="shin_l" value="0.1525"/>
+    <xacro:property name="leg_m" value="0.5"/>
+    <xacro:property name="leg_r" value="0.02"/>
+    <material name="gray"><color rgba="0.5 0.5 0.5 1"/></material>
+    <material name="black"><color rgba="0.1 0.1 0.1 1"/></material>
     <xacro:macro name="box_inertia" params="m x y z">
         <inertial>
             <mass value="${m}"/>
-            <inertia ixx="0.1" ixy="0" ixz="0" iyy="0.1" iyz="0" izz="0.1"/>
+            <inertia ixx="0.05" ixy="0" ixz="0" iyy="0.1" iyz="0" izz="0.1"/>
         </inertial>
     </xacro:macro>
@@ -19,94 +21,78 @@
         <inertial>
             <mass value="${m}"/>
-            <inertia ixx="0.01" ixy="0" ixz="0" iyy="0.1" iyz="0" izz="0.1"/>
+            <inertia ixx="0.015" ixy="0" ixz="0" iyy="0.015" iyz="0" izz="0.015"/>
         </inertial>
     </xacro:macro>
-    <material name="gray"><color rgba="0.5 0.5 0.5 1"/></material>
-    <material name="black"><color rgba="0.1 0.1 0.1 1"/></material>
-    <!-- BASE & TRUNK -->
+    <xacro:macro name="leg_inertia" params="m">
+        <inertial>
+            <mass value="${m}"/>
+            <inertia ixx="0.005" ixy="0" ixz="0" iyy="0.005" iyz="0" izz="0.005"/>
+        </inertial>
+    </xacro:macro>
     <link name="base_link"><visual><geometry><box size="0.01 0.01 0.01"/></geometry></visual></link>
-    <joint name="base_joint" type="fixed">
-        <parent link="base_link"/>
-        <child link="trunk"/>
-    </joint>
+    <joint name="base_joint" type="fixed"><parent link="base_link"/><child link="trunk"/></joint>
     <link name="trunk">
-        <visual>
-            <geometry><box size="${trunk_l} ${trunk_w} ${trunk_h}"/></geometry>
-            <material name="gray"/>
-        </visual>
-        <collision>
-            <geometry><box size="${trunk_l} ${trunk_w} ${trunk_h}"/></geometry>
-        </collision>
-        <xacro:box_inertia m="${trunk_m}" x="${trunk_l}" y="${trunk_w}" z="${trunk_h}"/>
+        <visual><geometry><box size="${trunk_l} ${trunk_w} ${trunk_h}"/></geometry><material name="gray"/></visual>
+        <collision><geometry><box size="${trunk_l} ${trunk_w} ${trunk_h}"/></geometry></collision>
+        <inertial>
+            <mass value="${trunk_m}"/>
+            <origin xyz="-0.05 0 0" rpy="0 0 0"/>
+            <inertia ixx="0.05" ixy="0" ixz="0" iyy="0.1" iyz="0" izz="0.1"/>
+        </inertial>
     </link>
-    <!-- LEG MACRO -->
     <xacro:macro name="dog_leg" params="prefix side_x side_y">
         <!-- HIP -->
         <joint name="${prefix}_hip_joint" type="revolute">
-            <parent link="trunk"/>
-            <child link="${prefix}_hip"/>
+            <parent link="trunk"/> <child link="${prefix}_hip"/>
             <origin xyz="${side_x * trunk_l/2} ${side_y * trunk_w/2} 0" rpy="0 0 0"/>
-            <axis xyz="1 0 0"/>
-            <limit lower="-0.7" upper="0.7" effort="50" velocity="5"/>
-            <dynamics damping="1.0" friction="0.5"/>
+            <axis xyz="1 0 0"/> <limit lower="-0.8" upper="0.8" effort="20" velocity="20"/>
         </joint>
         <link name="${prefix}_hip">
-            <visual>
-                <origin xyz="0 ${side_y * 0.05} 0"/>
-                <geometry><box size="0.1 0.1 0.1"/></geometry>
-                <material name="black"/>
-            </visual>
-            <!-- <collision> ... </collision> -->
-            <xacro:box_inertia m="0.5" x="0.1" y="0.1" z="0.1"/>
+            <visual><geometry><box size="0.05 0.05 0.05"/></geometry><material name="black"/></visual>
+            <xacro:leg_inertia m="0.2"/>
         </link>
         <!-- THIGH -->
         <joint name="${prefix}_thigh_joint" type="revolute">
-            <parent link="${prefix}_hip"/>
-            <child link="${prefix}_thigh"/>
-            <origin xyz="0 ${side_y * 0.05} 0" rpy="0 0 0"/>
-            <axis xyz="0 1 0"/>
-            <limit lower="-1.5" upper="1.5" effort="50" velocity="5"/>
-            <dynamics damping="1.0" friction="0.5"/>
+            <parent link="${prefix}_hip"/> <child link="${prefix}_thigh"/>
+            <origin xyz="0 ${side_y * hip_l} 0" rpy="0 0 0"/>
+            <axis xyz="0 1 0"/> <limit lower="-1.0" upper="4.0" effort="20" velocity="20"/>
         </joint>
         <link name="${prefix}_thigh">
             <visual>
-                <origin xyz="0 0 ${-thigh_l/2}" rpy="0 0 0"/>
-                <geometry><cylinder radius="${leg_r}" length="${thigh_l}"/></geometry>
-                <material name="gray"/>
+                <origin xyz="0 0 ${-thigh_l/2}"/><geometry><cylinder radius="${leg_r}" length="${thigh_l}"/></geometry><material name="gray"/>
             </visual>
             <collision>
-                <origin xyz="0 0 ${-thigh_l/2}" rpy="0 0 0"/>
-                <geometry><cylinder radius="0.015" length="${thigh_l - 0.04}"/></geometry>
+                <origin xyz="0 0 ${-thigh_l/2}"/><geometry><cylinder radius="${leg_r}" length="${thigh_l - 0.04}"/></geometry>
             </collision>
-            <xacro:cylinder_inertia m="${leg_m}" r="${leg_r}" h="${thigh_l}"/>
+            <xacro:leg_inertia m="${leg_m}"/>
         </link>
         <!-- SHIN -->
         <joint name="${prefix}_shin_joint" type="revolute">
-            <parent link="${prefix}_thigh"/>
-            <child link="${prefix}_shin"/>
+            <parent link="${prefix}_thigh"/> <child link="${prefix}_shin"/>
             <origin xyz="0 0 ${-thigh_l}" rpy="0 0 0"/>
-            <axis xyz="0 1 0"/>
-            <limit lower="-2.5" upper="0.0" effort="50" velocity="5"/>
-            <dynamics damping="1.0" friction="0.5"/>
+            <axis xyz="0 1 0"/> <limit lower="-4.0" upper="-0.5" effort="20" velocity="20"/>
         </joint>
         <link name="${prefix}_shin">
             <visual>
-                <origin xyz="0 0 ${-shin_l/2}" rpy="0 0 0"/>
-                <geometry><cylinder radius="${leg_r*0.8}" length="${shin_l}"/></geometry>
-                <material name="black"/>
+                <origin xyz="0 0 ${-shin_l/2}"/><geometry><cylinder radius="${leg_r*0.8}" length="${shin_l}"/></geometry><material name="black"/>
             </visual>
             <collision>
-                <origin xyz="0 0 ${-shin_l}" rpy="0 0 0"/>
-                <geometry><sphere radius="0.04"/></geometry>
+                <origin xyz="0 0 ${-shin_l}"/>
+                <geometry><sphere radius="0.03"/></geometry>
                 <surface>
                     <friction>
                         <ode>
-                            <mu>200.0</mu>
-                            <mu2>200.0</mu2>
+                            <mu>100.0</mu>
+                            <mu2>100.0</mu2>
                             <fdir1>1 0 0</fdir1>
                         </ode>
                     </friction>
                     <contact>
-                        <ode><kp>100000.0</kp><kd>1000.0</kd><min_depth>0.001</min_depth></ode>
+                        <ode>
+                            <kp>500000.0</kp>
+                            <kd>100.0</kd>
+                            <minDepth>0.002</minDepth>
+                            <maxVel>0.0</maxVel>
+                        </ode>
                     </contact>
                 </surface>
@@ -121,16 +107,19 @@
     <ros2_control name="GazeboSystem" type="system">
         <hardware><plugin>gazebo_ros2_control/GazeboSystem</plugin></hardware>
-        <joint name="front_left_hip_joint"><command_interface name="position"/><state_interface name="velocity"/><state_interface name="position"><param name="initial_value">0.0</param></state_interface></joint>
-        <joint name="front_left_thigh_joint"><command_interface name="position"/><state_interface name="velocity"/><state_interface name="position"><param name="initial_value">0.9</param></state_interface></joint>
-        <joint name="front_left_shin_joint"><command_interface name="position"/><state_interface name="velocity"/><state_interface name="position"><param name="initial_value">-1.8</param></state_interface></joint>
-        <joint name="front_right_hip_joint"><command_interface name="position"/><state_interface name="velocity"/><state_interface name="position"><param name="initial_value">0.0</param></state_interface></joint>
-        <joint name="front_right_thigh_joint"><command_interface name="position"/><state_interface name="velocity"/><state_interface name="position"><param name="initial_value">0.9</param></state_interface></joint>
-        <joint name="front_right_shin_joint"><command_interface name="position"/><state_interface name="velocity"/><state_interface name="position"><param name="initial_value">-1.8</param></state_interface></joint>
-        <joint name="rear_left_hip_joint"><command_interface name="position"/><state_interface name="velocity"/><state_interface name="position"><param name="initial_value">0.0</param></state_interface></joint>
-        <joint name="rear_left_thigh_joint"><command_interface name="position"/><state_interface name="velocity"/><state_interface name="position"><param name="initial_value">0.9</param></state_interface></joint>
-        <joint name="rear_left_shin_joint"><command_interface name="position"/><state_interface name="velocity"/><state_interface name="position"><param name="initial_value">-1.8</param></state_interface></joint>
-        <joint name="rear_right_hip_joint"><command_interface name="position"/><state_interface name="velocity"/><state_interface name="position"><param name="initial_value">0.0</param></state_interface></joint>
-        <joint name="rear_right_thigh_joint"><command_interface name="position"/><state_interface name="velocity"/><state_interface name="position"><param name="initial_value">0.9</param></state_interface></joint>
-        <joint name="rear_right_shin_joint"><command_interface name="position"/><state_interface name="velocity"/><state_interface name="position"><param name="initial_value">-1.8</param></state_interface></joint>
+        <xacro:macro name="ctrl_joint" params="name thigh_val shin_val">
+            <joint name="${name}_hip_joint">
+                <command_interface name="position"/><state_interface name="velocity"/><state_interface name="position"><param name="initial_value">0.0</param></state_interface>
+            </joint>
+            <joint name="${name}_thigh_joint">
+                <command_interface name="position"/><state_interface name="velocity"/><state_interface name="position"><param name="initial_value">${thigh_val}</param></state_interface>
+            </joint>
+            <joint name="${name}_shin_joint">
+                <command_interface name="position"/><state_interface name="velocity"/><state_interface name="position"><param name="initial_value">${shin_val}</param></state_interface>
+            </joint>
+        </xacro:macro>
+        <xacro:ctrl_joint name="front_left" thigh_val="0.7" shin_val="-1.4"/>
+        <xacro:ctrl_joint name="front_right" thigh_val="0.7" shin_val="-1.4"/>
+        <xacro:ctrl_joint name="rear_left" thigh_val="0.7" shin_val="-1.4"/>
+        <xacro:ctrl_joint name="rear_right" thigh_val="0.7" shin_val="-1.4"/>
     </ros2_control>
     <gazebo>
@@ -139,18 +128,3 @@
         </plugin>
     </gazebo>
-    <xacro:macro name="foot_physics" params="prefix">
-        <gazebo reference="${prefix}_shin">
-            <mu1>10.0</mu1>
-            <mu2>10.0</mu2>
-            <kp>1000000.0</kp>
-            <kd>1.0</kd>
-            <maxVel>0.0</maxVel>
-            <minDepth>0.002</minDepth>
-            <material>Gazebo/Black</material>
-        </gazebo>
-    </xacro:macro>
-    <xacro:foot_physics prefix="front_left"/>
-    <xacro:foot_physics prefix="front_right"/>
-    <xacro:foot_physics prefix="rear_left"/>
-    <xacro:foot_physics prefix="rear_right"/>
 </robot>

Commit message: вроде как ходит, но когда просто стоит скользит назад

File: src/dog_description/urdf/dog.urdf.xacro (robot description, xacro)
@@ -50,4 +50,5 @@
         <link name="${prefix}_hip">
             <visual><geometry><box size="0.05 0.05 0.05"/></geometry><material name="black"/></visual>
+            <collision><geometry><box size="0.001 0.001 0.001"/></geometry></collision>
             <xacro:leg_inertia m="0.2"/>
         </link>
@@ -63,5 +64,6 @@
             </visual>
             <collision>
-                <origin xyz="0 0 ${-thigh_l/2}"/><geometry><cylinder radius="${leg_r}" length="${thigh_l - 0.04}"/></geometry>
+                <origin xyz="0 0 ${-thigh_l/2}"/>
+                <geometry><cylinder radius="0.001" length="0.001"/></geometry>
             </collision>
             <xacro:leg_inertia m="${leg_m}"/>
@@ -79,24 +81,21 @@
             <collision>
                 <origin xyz="0 0 ${-shin_l}"/>
-                <geometry><sphere radius="0.03"/></geometry>
+                <geometry><sphere radius="0.04"/></geometry>
                 <surface>
                     <friction>
                         <ode>
-                            <mu>100.0</mu>
-                            <mu2>100.0</mu2>
-                            <fdir1>1 0 0</fdir1>
+                            <mu>200.0</mu> <mu2>200.0</mu2>
                         </ode>
                     </friction>
                     <contact>
                         <ode>
-                            <kp>500000.0</kp>
-                            <kd>100.0</kd>
-                            <minDepth>0.002</minDepth>
-                            <maxVel>0.0</maxVel>
+                            <kp>1000000.0</kp>
+                            <kd>10.0</kd>
+                            <minDepth>0.001</minDepth>
                         </ode>
                     </contact>
                 </surface>
             </collision>
-            <xacro:cylinder_inertia m="${leg_m}" r="${leg_r*0.8}" h="${shin_l}"/>
+            <xacro:leg_inertia m="${leg_m}"/>
         </link>
     </xacro:macro>
@@ -118,8 +117,8 @@
             </joint>
         </xacro:macro>
-        <xacro:ctrl_joint name="front_left" thigh_val="0.7" shin_val="-1.4"/>
-        <xacro:ctrl_joint name="front_right" thigh_val="0.7" shin_val="-1.4"/>
-        <xacro:ctrl_joint name="rear_left" thigh_val="0.7" shin_val="-1.4"/>
-        <xacro:ctrl_joint name="rear_right" thigh_val="0.7" shin_val="-1.4"/>
+        <xacro:ctrl_joint name="front_left" thigh_val="0.1" shin_val="-0.2"/>
+        <xacro:ctrl_joint name="front_right" thigh_val="0.1" shin_val="-0.2"/>
+        <xacro:ctrl_joint name="rear_left" thigh_val="0.1" shin_val="-0.2"/>
+        <xacro:ctrl_joint name="rear_right" thigh_val="0.1" shin_val="-0.2"/>
     </ros2_control>
     <gazebo>

Commit message: хоть чет

File: src/dog_description/urdf/dog.urdf.xacro (robot description, xacro)
@@ -42,21 +42,30 @@
     </link>
     <xacro:macro name="dog_leg" params="prefix side_x side_y">
-        <!-- HIP -->
+        <!-- HIP JOINT -->
         <joint name="${prefix}_hip_joint" type="revolute">
             <parent link="trunk"/> <child link="${prefix}_hip"/>
             <origin xyz="${side_x * trunk_l/2} ${side_y * trunk_w/2} 0" rpy="0 0 0"/>
-            <axis xyz="1 0 0"/> <limit lower="-0.8" upper="0.8" effort="20" velocity="20"/>
+            <axis xyz="1 0 0"/>
+            <limit lower="-0.8" upper="0.8" effort="20" velocity="20"/>
+            <dynamics damping="0.5" friction="0.5"/>
         </joint>
+        <gazebo reference="${prefix}_hip_joint">
+            <implicitSpringDamper>true</implicitSpringDamper>
+        </gazebo>
         <link name="${prefix}_hip">
             <visual><geometry><box size="0.05 0.05 0.05"/></geometry><material name="black"/></visual>
-            <collision><geometry><box size="0.001 0.001 0.001"/></geometry></collision>
             <xacro:leg_inertia m="0.2"/>
         </link>
-        <!-- THIGH -->
+        <!-- THIGH JOINT -->
         <joint name="${prefix}_thigh_joint" type="revolute">
             <parent link="${prefix}_hip"/> <child link="${prefix}_thigh"/>
             <origin xyz="0 ${side_y * hip_l} 0" rpy="0 0 0"/>
-            <axis xyz="0 1 0"/> <limit lower="-1.0" upper="4.0" effort="20" velocity="20"/>
+            <axis xyz="0 1 0"/>
+            <limit lower="-1.0" upper="4.0" effort="20" velocity="20"/>
+            <dynamics damping="0.5" friction="0.5"/>
         </joint>
+        <gazebo reference="${prefix}_thigh_joint">
+            <implicitSpringDamper>true</implicitSpringDamper>
+        </gazebo>
         <link name="${prefix}_thigh">
             <visual>
@@ -64,15 +73,19 @@
             </visual>
             <collision>
-                <origin xyz="0 0 ${-thigh_l/2}"/>
-                <geometry><cylinder radius="0.001" length="0.001"/></geometry>
+                <origin xyz="0 0 ${-thigh_l/2}"/><geometry><cylinder radius="${leg_r}" length="${thigh_l - 0.04}"/></geometry>
             </collision>
             <xacro:leg_inertia m="${leg_m}"/>
         </link>
-        <!-- SHIN -->
+        <!-- SHIN JOINT -->
         <joint name="${prefix}_shin_joint" type="revolute">
             <parent link="${prefix}_thigh"/> <child link="${prefix}_shin"/>
             <origin xyz="0 0 ${-thigh_l}" rpy="0 0 0"/>
-            <axis xyz="0 1 0"/> <limit lower="-4.0" upper="-0.5" effort="20" velocity="20"/>
+            <axis xyz="0 1 0"/>
+            <limit lower="-4.0" upper="-0.5" effort="20" velocity="20"/>
+            <dynamics damping="0.5" friction="0.5"/>
         </joint>
+        <gazebo reference="${prefix}_shin_joint">
+            <implicitSpringDamper>true</implicitSpringDamper>
+        </gazebo>
         <link name="${prefix}_shin">
             <visual>
@@ -81,17 +94,11 @@
             <collision>
                 <origin xyz="0 0 ${-shin_l}"/>
-                <geometry><sphere radius="0.04"/></geometry>
+                <geometry><sphere radius="0.03"/></geometry>
                 <surface>
                     <friction>
-                        <ode>
-                            <mu>200.0</mu> <mu2>200.0</mu2>
-                        </ode>
+                        <ode><mu>200.0</mu><mu2>200.0</mu2></ode>
                     </friction>
                     <contact>
-                        <ode>
-                            <kp>1000000.0</kp>
-                            <kd>10.0</kd>
-                            <minDepth>0.001</minDepth>
-                        </ode>
+                        <ode><kp>1000000.0</kp><kd>100.0</kd><minDepth>0.001</minDepth></ode>
                     </contact>
                 </surface>
@@ -117,8 +124,8 @@
             </joint>
         </xacro:macro>
-        <xacro:ctrl_joint name="front_left" thigh_val="0.1" shin_val="-0.2"/>
-        <xacro:ctrl_joint name="front_right" thigh_val="0.1" shin_val="-0.2"/>
-        <xacro:ctrl_joint name="rear_left" thigh_val="0.1" shin_val="-0.2"/>
-        <xacro:ctrl_joint name="rear_right" thigh_val="0.1" shin_val="-0.2"/>
+        <xacro:ctrl_joint name="front_left" thigh_val="0.5" shin_val="-1.1"/>
+        <xacro:ctrl_joint name="front_right" thigh_val="0.5" shin_val="-1.1"/>
+        <xacro:ctrl_joint name="rear_left" thigh_val="0.5" shin_val="-1.1"/>
+        <xacro:ctrl_joint name="rear_right" thigh_val="0.5" shin_val="-1.1"/>
     </ros2_control>
     <gazebo>

Commit message: вроде рабочая походка вперед, начало телеопа

File: src/dog_description/urdf/dog.urdf.xacro (robot description, xacro)
@@ -48,5 +48,4 @@
             <axis xyz="1 0 0"/>
             <limit lower="-0.8" upper="0.8" effort="20" velocity="20"/>
-            <dynamics damping="0.5" friction="0.5"/>
         </joint>
         <gazebo reference="${prefix}_hip_joint">
@@ -63,5 +62,4 @@
             <axis xyz="0 1 0"/>
             <limit lower="-1.0" upper="4.0" effort="20" velocity="20"/>
-            <dynamics damping="0.5" friction="0.5"/>
         </joint>
         <gazebo reference="${prefix}_thigh_joint">
@@ -83,5 +81,4 @@
             <axis xyz="0 1 0"/>
             <limit lower="-4.0" upper="-0.5" effort="20" velocity="20"/>
-            <dynamics damping="0.5" friction="0.5"/>
         </joint>
         <gazebo reference="${prefix}_shin_joint">
@@ -97,8 +94,16 @@
                 <surface>
                     <friction>
-                        <ode><mu>200.0</mu><mu2>200.0</mu2></ode>
+                        <ode>
+                            <mu>1.0</mu>
+                            <mu2>1.0</mu2>
+                        </ode>
                     </friction>
                     <contact>
-                        <ode><kp>1000000.0</kp><kd>100.0</kd><minDepth>0.001</minDepth></ode>
+                        <ode>
+                            <kp>500000.0</kp>
+                            <kd>100.0</kd>
+                            <minDepth>0.003</minDepth>
+                            <maxVel>0.0</maxVel>
+                        </ode>
                     </contact>
                 </surface>
