Commit message: переделанная архитектура, rviz есть но летает собак

File: src/dog_description/urdf/dog.urdf.xacro (robot description, xacro)
@@ -1,4 +1,5 @@
 <?xml version="1.0"?>
 <robot xmlns:xacro="http://www.ros.org/wiki/xacro" name="dog">
+    <!-- ==================== PROPERTIES ==================== -->
     <xacro:property name="trunk_l" value="0.475"/>
     <xacro:property name="trunk_w" value="0.18"/>
@@ -6,136 +7,194 @@
     <xacro:property name="trunk_m" value="6.0"/>
     <xacro:property name="hip_l" value="0.06"/>
+    <xacro:property name="hip_m" value="0.2"/>
+    <xacro:property name="hip_r" value="0.02"/>
     <xacro:property name="thigh_l" value="0.144"/>
     <xacro:property name="shin_l" value="0.1525"/>
-    <xacro:property name="leg_m" value="0.5"/>
+    <xacro:property name="leg_m" value="0.6"/>
     <xacro:property name="leg_r" value="0.02"/>
-    <material name="gray"><color rgba="0.5 0.5 0.5 1"/></material>
+    <xacro:property name="foot_r" value="0.025"/>
+    <!-- Начальная поза стойки: IK(x=0, z=-0.22) -->
+    <!-- thigh=0.76 rad, shin=-1.47 rad => нога опущена на 0.22м ниже бедра -->
+    <xacro:property name="init_thigh" value="0.76"/>
+    <xacro:property name="init_shin" value="-1.47"/>
+    <!-- ==================== MATERIALS ==================== -->
     <material name="black"><color rgba="0.1 0.1 0.1 1"/></material>
-    <xacro:macro name="box_inertia" params="m x y z">
+    <material name="grey"><color rgba="0.6 0.6 0.6 1"/></material>
+    <!-- ==================== INERTIA MACROS ==================== -->
+    <!-- Box inertia (CoM в центре box) -->
+    <xacro:macro name="box_inertia" params="m l w h">
         <inertial>
             <mass value="${m}"/>
-            <inertia ixx="0.05" ixy="0" ixz="0" iyy="0.1" iyz="0" izz="0.1"/>
+            <inertia ixx="${m/12*(w*w+h*h)}" ixy="0" ixz="0"
+                     iyy="${m/12*(l*l+h*h)}" iyz="0"
+                     izz="${m/12*(l*l+w*w)}"/>
         </inertial>
     </xacro:macro>
-    <xacro:macro name="cylinder_inertia" params="m r h">
+    <!-- Cylinder inertia со смещённым центром масс -->
+    <xacro:macro name="cylinder_inertia_offset" params="m r h ox oy oz">
         <inertial>
+            <origin xyz="${ox} ${oy} ${oz}"/>
             <mass value="${m}"/>
-            <inertia ixx="0.015" ixy="0" ixz="0" iyy="0.015" iyz="0" izz="0.015"/>
+            <inertia ixx="${m/12*(3*r*r+h*h)}" ixy="0" ixz="0"
+                     iyy="${m/12*(3*r*r+h*h)}" iyz="0"
+                     izz="${m*r*r/2}"/>
         </inertial>
     </xacro:macro>
-    <xacro:macro name="leg_inertia" params="m">
-        <inertial>
-            <mass value="${m}"/>
-            <inertia ixx="0.005" ixy="0" ixz="0" iyy="0.005" iyz="0" izz="0.005"/>
-        </inertial>
-    </xacro:macro>
-    <link name="base_link"><visual><geometry><box size="0.01 0.01 0.01"/></geometry></visual></link>
-    <joint name="base_joint" type="fixed"><parent link="base_link"/><child link="trunk"/></joint>
+    <!-- ==================== TRUNK ==================== -->
+    <link name="base_link">
+        <visual><geometry><box size="0.01 0.01 0.01"/></geometry></visual>
+    </link>
+    <joint name="base_joint" type="fixed">
+        <parent link="base_link"/><child link="trunk"/>
+    </joint>
     <link name="trunk">
-        <visual><geometry><box size="${trunk_l} ${trunk_w} ${trunk_h}"/></geometry><material name="gray"/></visual>
-        <collision><geometry><box size="${trunk_l} ${trunk_w} ${trunk_h}"/></geometry></collision>
-        <inertial>
-            <mass value="${trunk_m}"/>
-            <origin xyz="-0.05 0 0" rpy="0 0 0"/>
-            <inertia ixx="0.05" ixy="0" ixz="0" iyy="0.1" iyz="0" izz="0.1"/>
-        </inertial>
+        <visual>
+            <geometry><box size="${trunk_l} ${trunk_w} ${trunk_h}"/></geometry>
+            <material name="grey"/>
+        </visual>
+        <collision>
+            <geometry><box size="${trunk_l} ${trunk_w} ${trunk_h}"/></geometry>
+        </collision>
+        <xacro:box_inertia m="${trunk_m}" l="${trunk_l}" w="${trunk_w}" h="${trunk_h}"/>
     </link>
+    <!-- ==================== FOOT FRICTION MACRO ==================== -->
+    <xacro:macro name="foot_friction" params="prefix">
+        <gazebo reference="${prefix}_shin">
+            <mu1>1.5</mu1>
+            <mu2>1.5</mu2>
+            <kp>100000.0</kp>
+            <kd>100.0</kd>
+            <minDepth>0.001</minDepth>
+        </gazebo>
+    </xacro:macro>
+    <!-- ==================== LEG MACRO ==================== -->
     <xacro:macro name="dog_leg" params="prefix side_x side_y">
-        <!-- HIP JOINT -->
+        <!-- 1. HIP (Roll) -->
         <joint name="${prefix}_hip_joint" type="revolute">
             <parent link="trunk"/> <child link="${prefix}_hip"/>
             <origin xyz="${side_x * trunk_l/2} ${side_y * trunk_w/2} 0" rpy="0 0 0"/>
             <axis xyz="1 0 0"/>
-            <limit lower="-0.8" upper="0.8" effort="20" velocity="20"/>
+            <limit lower="-0.5" upper="0.5" effort="20" velocity="10"/>
+            <dynamics damping="1.0" friction="0.3"/>
         </joint>
-        <gazebo reference="${prefix}_hip_joint">
-            <implicitSpringDamper>true</implicitSpringDamper>
-        </gazebo>
         <link name="${prefix}_hip">
-            <visual><geometry><box size="0.05 0.05 0.05"/></geometry><material name="black"/></visual>
-            <xacro:leg_inertia m="0.2"/>
+            <visual>
+                <origin xyz="0 ${side_y * hip_l/2} 0" rpy="${pi/2} 0 0"/>
+                <geometry><cylinder radius="${hip_r}" length="${hip_l}"/></geometry>
+                <material name="black"/>
+            </visual>
+            <xacro:cylinder_inertia_offset m="${hip_m}" r="${hip_r}" h="${hip_l}"
+                ox="0" oy="${side_y * hip_l/2}" oz="0"/>
         </link>
-        <!-- THIGH JOINT -->
+        <!-- 2. THIGH (Pitch) -->
         <joint name="${prefix}_thigh_joint" type="revolute">
             <parent link="${prefix}_hip"/> <child link="${prefix}_thigh"/>
             <origin xyz="0 ${side_y * hip_l} 0" rpy="0 0 0"/>
             <axis xyz="0 1 0"/>
-            <limit lower="-1.0" upper="4.0" effort="20" velocity="20"/>
+            <limit lower="-0.5" upper="2.5" effort="20" velocity="10"/>
+            <dynamics damping="1.0" friction="0.3"/>
         </joint>
-        <gazebo reference="${prefix}_thigh_joint">
-            <implicitSpringDamper>true</implicitSpringDamper>
-        </gazebo>
         <link name="${prefix}_thigh">
             <visual>
-                <origin xyz="0 0 ${-thigh_l/2}"/><geometry><cylinder radius="${leg_r}" length="${thigh_l}"/></geometry><material name="gray"/>
+                <origin xyz="0 0 ${-thigh_l/2}"/>
+                <geometry><cylinder radius="${leg_r}" length="${thigh_l}"/></geometry>
+                <material name="grey"/>
             </visual>
             <collision>
-                <origin xyz="0 0 ${-thigh_l/2}"/><geometry><cylinder radius="${leg_r}" length="${thigh_l - 0.04}"/></geometry>
+                <origin xyz="0 0 ${-thigh_l/2}"/>
+                <geometry><cylinder radius="${leg_r}" length="${thigh_l - 0.04}"/></geometry>
             </collision>
-            <xacro:leg_inertia m="${leg_m}"/>
+            <xacro:cylinder_inertia_offset m="${leg_m}" r="${leg_r}" h="${thigh_l}"
+                ox="0" oy="0" oz="${-thigh_l/2}"/>
         </link>
-        <!-- SHIN JOINT -->
+        <!-- 3. SHIN (Pitch) -->
         <joint name="${prefix}_shin_joint" type="revolute">
             <parent link="${prefix}_thigh"/> <child link="${prefix}_shin"/>
             <origin xyz="0 0 ${-thigh_l}" rpy="0 0 0"/>
             <axis xyz="0 1 0"/>
-            <limit lower="-4.0" upper="-0.5" effort="20" velocity="20"/>
+            <limit lower="-2.7" upper="-0.3" effort="20" velocity="10"/>
+            <dynamics damping="1.0" friction="0.3"/>
         </joint>
-        <gazebo reference="${prefix}_shin_joint">
-            <implicitSpringDamper>true</implicitSpringDamper>
-        </gazebo>
         <link name="${prefix}_shin">
             <visual>
-                <origin xyz="0 0 ${-shin_l/2}"/><geometry><cylinder radius="${leg_r*0.8}" length="${shin_l}"/></geometry><material name="black"/>
+                <origin xyz="0 0 ${-shin_l/2}"/>
+                <geometry><cylinder radius="${leg_r*0.8}" length="${shin_l}"/></geometry>
+                <material name="black"/>
             </visual>
             <collision>
+                <origin xyz="0 0 ${-shin_l/2}"/>
+                <geometry><cylinder radius="${leg_r*0.8}" length="${shin_l}"/></geometry>
+            </collision>
+            <!-- Foot sphere -->
+            <collision>
                 <origin xyz="0 0 ${-shin_l}"/>
-                <geometry><sphere radius="0.03"/></geometry>
-                <surface>
-                    <friction>
-                        <ode>
-                            <mu>1.0</mu>
-                            <mu2>1.0</mu2>
-                        </ode>
-                    </friction>
-                    <contact>
-                        <ode>
-                            <kp>500000.0</kp>
-                            <kd>100.0</kd>
-                            <minDepth>0.003</minDepth>
-                            <maxVel>0.0</maxVel>
-                        </ode>
-                    </contact>
-                </surface>
+                <geometry><sphere radius="${foot_r}"/></geometry>
             </collision>
-            <xacro:leg_inertia m="${leg_m}"/>
+            <xacro:cylinder_inertia_offset m="${leg_m}" r="${leg_r*0.8}" h="${shin_l}"
+                ox="0" oy="0" oz="${-shin_l/2}"/>
         </link>
-    </xacro:macro>
+        <xacro:foot_friction prefix="${prefix}"/>
+    </xacro:macro>
+    <!-- ==================== INSTANTIATE LEGS ==================== -->
     <xacro:dog_leg prefix="front_left"  side_x="1"  side_y="1"/>
     <xacro:dog_leg prefix="front_right" side_x="1"  side_y="-1"/>
     <xacro:dog_leg prefix="rear_left"   side_x="-1" side_y="1"/>
     <xacro:dog_leg prefix="rear_right"  side_x="-1" side_y="-1"/>
+    <!-- ==================== ROS2 CONTROL ==================== -->
     <ros2_control name="GazeboSystem" type="system">
         <hardware><plugin>gazebo_ros2_control/GazeboSystem</plugin></hardware>
-        <xacro:macro name="ctrl_joint" params="name thigh_val shin_val">
+        <xacro:macro name="init_pos" params="name t s">
             <joint name="${name}_hip_joint">
-                <command_interface name="position"/><state_interface name="velocity"/><state_interface name="position"><param name="initial_value">0.0</param></state_interface>
+                <state_interface name="position"><param name="initial_value">0.0</param></state_interface>
+                <command_interface name="position"/>
+                <state_interface name="velocity"/>
             </joint>
             <joint name="${name}_thigh_joint">
-                <command_interface name="position"/><state_interface name="velocity"/><state_interface name="position"><param name="initial_value">${thigh_val}</param></state_interface>
+                <state_interface name="position"><param name="initial_value">${t}</param></state_interface>
+                <command_interface name="position"/>
+                <state_interface name="velocity"/>
             </joint>
             <joint name="${name}_shin_joint">
-                <command_interface name="position"/><state_interface name="velocity"/><state_interface name="position"><param name="initial_value">${shin_val}</param></state_interface>
+                <state_interface name="position"><param name="initial_value">${s}</param></state_interface>
+                <command_interface name="position"/>
+                <state_interface name="velocity"/>
             </joint>
         </xacro:macro>
-        <xacro:ctrl_joint name="front_left" thigh_val="0.5" shin_val="-1.1"/>
-        <xacro:ctrl_joint name="front_right" thigh_val="0.5" shin_val="-1.1"/>
-        <xacro:ctrl_joint name="rear_left" thigh_val="0.5" shin_val="-1.1"/>
-        <xacro:ctrl_joint name="rear_right" thigh_val="0.5" shin_val="-1.1"/>
+        <xacro:init_pos name="front_left"  t="${init_thigh}" s="${init_shin}"/>
+        <xacro:init_pos name="front_right" t="${init_thigh}" s="${init_shin}"/>
+        <xacro:init_pos name="rear_left"   t="${init_thigh}" s="${init_shin}"/>
+        <xacro:init_pos name="rear_right"  t="${init_thigh}" s="${init_shin}"/>
     </ros2_control>
+    <!-- ==================== GAZEBO PLUGINS ==================== -->
     <gazebo>
         <plugin name="gazebo_ros2_control" filename="libgazebo_ros2_control.so">
-            <parameters>$(find dog_controllers)/config/controllers.yaml</parameters>
+            <parameters>$(find dog_bringup)/config/controllers.yaml</parameters>
         </plugin>
     </gazebo>
+    <!-- IMU Sensor on trunk -->
+    <gazebo reference="trunk">
+        <sensor name="imu_sensor" type="imu">
+            <always_on>true</always_on>
+            <update_rate>100</update_rate>
+            <imu>
+                <angular_velocity>
+                    <x><noise type="gaussian"><mean>0.0</mean><stddev>0.0002</stddev></noise></x>
+                    <y><noise type="gaussian"><mean>0.0</mean><stddev>0.0002</stddev></noise></y>
+                    <z><noise type="gaussian"><mean>0.0</mean><stddev>0.0002</stddev></noise></z>
+                </angular_velocity>
+                <linear_acceleration>
+                    <x><noise type="gaussian"><mean>0.0</mean><stddev>0.017</stddev></noise></x>
+                    <y><noise type="gaussian"><mean>0.0</mean><stddev>0.017</stddev></noise></y>
+                    <z><noise type="gaussian"><mean>0.0</mean><stddev>0.017</stddev></noise></z>
+                </linear_acceleration>
+            </imu>
+            <plugin name="imu_plugin" filename="libgazebo_ros_imu_sensor.so">
+                <ros>
+                    <remapping>~/out:=/imu/data</remapping>
+                </ros>
+                <initial_orientation_as_reference>false</initial_orientation_as_reference>
+                <frame_name>trunk</frame_name>
+            </plugin>
+        </sensor>
+    </gazebo>
 </robot>

Commit message: дрожание, верные meshes

File: src/dog_description/urdf/dog.urdf.xacro (robot description, xacro)
@@ -74,5 +74,5 @@
         <link name="${prefix}_shin">
             <visual>
-                <origin xyz="0 0 0" rpy="-1.5707963 0 0"/>
+                <origin xyz="-0.025 0 -0.03" rpy="-1.5707963 0 0"/>
                 <geometry><mesh filename="package://dog_description/meshes/leg11.STL" scale="0.001 0.001 0.001"/></geometry>
                 <material name="black"/>
@@ -83,8 +83,5 @@
                 <surface>
                     <friction>
-                        <ode>
-                            <mu>1.0</mu>
-                            <mu2>1.0</mu2>
-                        </ode>
+                        <ode><mu>1.0</mu><mu2>1.0</mu2></ode>
                     </friction>
                     <contact>
@@ -100,4 +97,12 @@
             <xacro:leg_inertia m="${leg_m}"/>
         </link>
+        <gazebo reference="${prefix}_shin">
+            <mu1>1.0</mu1>
+            <mu2>1.0</mu2>
+            <kp>500000</kp>
+            <kd>100</kd>
+            <minDepth>0.003</minDepth>
+            <maxVel>0</maxVel>
+        </gazebo>
     </xacro:macro>
     <xacro:dog_leg prefix="front_left"  side_x="1"  side_y="1"/>

Commit message: вроде норм работает алгоритм походки но из-за скольжения на месте, скольжение в симе, readme update

File: src/dog_description/urdf/dog.urdf.xacro (robot description, xacro)
@@ -58,7 +58,5 @@
                 <material name="gray"/>
             </visual>
-            <collision>
-                <origin xyz="0 0 ${-thigh_l/2}"/><geometry><cylinder radius="${leg_r}" length="${thigh_l - 0.04}"/></geometry>
-            </collision>
+            <!-- No collision on thigh - only foot sphere contacts ground -->
             <xacro:leg_inertia m="${leg_m}"/>
         </link>
@@ -81,17 +79,4 @@
                 <origin xyz="0 0 ${-shin_l}"/>
                 <geometry><sphere radius="0.03"/></geometry>
-                <surface>
-                    <friction>
-                        <ode><mu>5.0</mu><mu2>5.0</mu2></ode>
-                    </friction>
-                    <contact>
-                        <ode>
-                            <kp>500000.0</kp>
-                            <kd>100.0</kd>
-                            <minDepth>0.003</minDepth>
-                            <maxVel>0.0</maxVel>
-                        </ode>
-                    </contact>
-                </surface>
             </collision>
             <xacro:leg_inertia m="${leg_m}"/>
@@ -109,4 +94,7 @@
                 <state_interface name="velocity"/>
                 <state_interface name="position"><param name="initial_value">0.0</param></state_interface>
+                <param name="pos_kp">20.0</param>
+                <param name="pos_ki">0.0</param>
+                <param name="pos_kd">5.0</param>
             </joint>
             <joint name="${name}_thigh_joint">
@@ -114,4 +102,7 @@
                 <state_interface name="velocity"/>
                 <state_interface name="position"><param name="initial_value">${thigh_val}</param></state_interface>
+                <param name="pos_kp">20.0</param>
+                <param name="pos_ki">0.0</param>
+                <param name="pos_kd">5.0</param>
             </joint>
             <joint name="${name}_shin_joint">
@@ -119,4 +110,7 @@
                 <state_interface name="velocity"/>
                 <state_interface name="position"><param name="initial_value">${shin_val}</param></state_interface>
+                <param name="pos_kp">20.0</param>
+                <param name="pos_ki">0.0</param>
+                <param name="pos_kd">5.0</param>
             </joint>
         </xacro:macro>
@@ -129,4 +123,13 @@
         <plugin name="gazebo_ros2_control" filename="libgazebo_ros2_control.so">
             <parameters>$(find dog_bringup)/config/controllers.yaml</parameters>
+        </plugin>
+    </gazebo>
+    <!-- Ground truth position monitor - publish base_link pose in world frame -->
+    <gazebo>
+        <plugin name="p3d_base_controller" filename="libgazebo_ros_p3d.so">
+            <ros><remapping>odom:=/ground_truth/state</remapping></ros>
+            <frame_name>world</frame_name>
+            <body_name>base_link</body_name>
+            <update_rate>50</update_rate>
         </plugin>
     </gazebo>

Commit message: скользит, верный trot

File: src/dog_description/urdf/dog.urdf.xacro (robot description, xacro)
@@ -35,8 +35,5 @@
             <axis xyz="1 0 0"/>
             <limit lower="-1.0" upper="1.0" effort="20" velocity="20"/>
-        </joint>
-        <gazebo reference="${prefix}_hip_joint">
-            <implicitSpringDamper>true</implicitSpringDamper>
-        </gazebo>
+                    </joint>
         <link name="${prefix}_hip">
             <visual><geometry><box size="0.05 0.05 0.05"/></geometry><material name="black"/></visual>
@@ -48,8 +45,5 @@
             <axis xyz="0 1 0"/>
             <limit lower="-1.0" upper="4.0" effort="20" velocity="20"/>
-        </joint>
-        <gazebo reference="${prefix}_thigh_joint">
-            <implicitSpringDamper>true</implicitSpringDamper>
-        </gazebo>
+                    </joint>
         <link name="${prefix}_thigh">
             <visual>
@@ -66,8 +60,5 @@
             <axis xyz="0 1 0"/>
             <limit lower="-4.0" upper="-0.1" effort="20" velocity="20"/>
-        </joint>
-        <gazebo reference="${prefix}_shin_joint">
-            <implicitSpringDamper>true</implicitSpringDamper>
-        </gazebo>
+                    </joint>
         <link name="${prefix}_shin">
             <visual>
@@ -94,7 +85,4 @@
                 <state_interface name="velocity"/>
                 <state_interface name="position"><param name="initial_value">0.0</param></state_interface>
-                <param name="pos_kp">20.0</param>
-                <param name="pos_ki">0.0</param>
-                <param name="pos_kd">5.0</param>
             </joint>
             <joint name="${name}_thigh_joint">
@@ -102,7 +90,4 @@
                 <state_interface name="velocity"/>
                 <state_interface name="position"><param name="initial_value">${thigh_val}</param></state_interface>
-                <param name="pos_kp">20.0</param>
-                <param name="pos_ki">0.0</param>
-                <param name="pos_kd">5.0</param>
             </joint>
             <joint name="${name}_shin_joint">
@@ -110,7 +95,4 @@
                 <state_interface name="velocity"/>
                 <state_interface name="position"><param name="initial_value">${shin_val}</param></state_interface>
-                <param name="pos_kp">20.0</param>
-                <param name="pos_ki">0.0</param>
-                <param name="pos_kd">5.0</param>
             </joint>
         </xacro:macro>
